File: boards/lt3557-boost-converter/lt3557-boost-converter.kicad_pcb (KiCad board)
At the start: 2 copper layers, 40.6 x 55.2 mm, 26 parts, among them P1 Enable, P2 BAT IN, P3 24V OUT, Q1 FDB86566, U1 LT3757

Commit message: lt3557-boost-converter: silkscreen
Other:
- board text added: "RX-VIPER LT3757 8V to 24V 240W Boost © Raphael Lehmann"
Changed lines of the file:
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@@
     (links 138)
     (no_connects 1)
-    (area 45.634 29.886 106.91 96.68)
+    (area 49.454999 30.404999 90.245001 85.800001)
     (thickness 1.6)
-    (drawings 6)
+    (drawings 9)
     (tracks 661)
     (zones 0)
@@
   )
   (setup
-    (last_trace_width 1)
+    (last_trace_width 0.25)
     (user_trace_width 0.25)
     (user_trace_width 0.35)
@@
       (effects (font (size 1 1) (thickness 0.15)))
     )
-    (fp_text value "BAT IN" (at 0 5.08) (layer F.Fab)
+    (fp_text value "BAT IN" (at -6.1595 -0.762 270) (layer F.SilkS)
       (effects (font (size 1 1) (thickness 0.15)))
     )
@@
       (effects (font (size 1 1) (thickness 0.15)))
     )
-    (fp_text value "24V OUT" (at 0 5.08 90) (layer F.Fab)
+    (fp_text value "24V OUT" (at -6.858 1.27 360) (layer F.SilkS)
       (effects (font (size 1 1) (thickness 0.15)))
     )
@@
     (descr "Mounting Hole 3.2mm, no annular, M3, DIN965")
     (tags "mounting hole 3.2mm no annular m3 din965")
-    (fp_text reference REF** (at 0 -3.8) (layer F.SilkS)
+    (fp_text reference REF** (at 0 -3.8) (layer F.SilkS) hide
       (effects (font (size 1 1) (thickness 0.15)))
     )
@@
     (fp_circle (center 0 0) (end 3.05 0) (layer F.CrtYd) (width 0.05))
     (pad 1 np_thru_hole circle (at 0 0) (size 3.2 3.2) (drill 3.2) (layers *.Cu *.Mask F.SilkS))
+  )
+  (gr_text "RX-VIPER\nLT3757\n8V to 24V\n240W Boost\n© Raphael\nLehmann" (at 71.1835 59.6265 90) (layer B.SilkS)
+    (effects (font (size 1.5 1.5) (thickness 0.2)) (justify mirror))
+  )
+  (gr_text "RX-VIPER\nLT3757\n8V to 24V\n240W Boost\n© Raphael\nLehmann" (at 55.3085 43.8785 180) (layer F.SilkS)
+    (effects (font (size 0.8 0.8) (thickness 0.15)))
+  )
+  (gr_text "RX-VIPER\nLT3757\n8V to 24V\n240W Boost\n© Raphael\nLehmann" (at 55.9435 62.103) (layer F.SilkS)
+    (effects (font (size 0.8 0.8) (thickness 0.15)))
   )
   (dimension 54.61 (width 0.3) (layer Dwgs.User)
@@
     )
   )
-  (zone (net 2) (net_name GND) (layer B.Mask) (hatch edge 0.508)
+  (zone (net 0) (net_name "") (layer B.Mask) (hatch edge 0.508)
     (priority 4)
     (connect_pads yes (clearance 0.3))

Commit message: lt3757-board: fix diode polarity in schematic and layout
Parts:
- moved D1 0.72 mm to (83.8, 75.0), turned to 180 degrees
Connections:
- D1 pad 1: /LT3757/24V_OUT -> /LT3757/L_D_FET
- D1 pad 2: /LT3757/L_D_FET -> /LT3757/24V_OUT
- D1 pad 3: (no net) -> /LT3757/L_D_FET
Routing:
- net /LT3757/24V_OUT: track 140.7 -> 115.0 mm, vias 52 -> 36
- net /LT3757/L_D_FET: track 54.0 -> 76.1 mm, vias 21 -> 43
