File: boards/mainboard/mainboard.sch (KiCad schematic (older format))
At the start: 25 parts, among them J101 Powerboard <-> Mainboard, J102 Probe position sensors, J103 Camera board, P101 Temperature, P102 Pressure, SW101 SW_PUSH, SW102 SW_PUSH, U101 LM1117-3.3

Commit message: [mainboard] add encoder subschematic with differential receivers and filters; add ds26lv32at.lib
Parts:
- removed J102: Probe position sensors, symbol DB9_FEMALE
Changed lines of the file:
@@
 LIBS:ltc2984
 LIBS:DB
+LIBS:ds26lv32at
 LIBS:mainboard-cache
 EELAYER 25 0
@@
 $Descr A4 11693 8268
 encoding utf-8
-Sheet 1 11
+Sheet 1 12
 Title "Mainboard overview"
 Date "2017-03-14"
-Rev "10"
+Rev "11"
 Comp "VIPER"
 Comment1 ""
@@
 $EndComp
 $Comp
-L GND #PWR113
+L GND #PWR110
 U 1 1 588947DC
 P 5500 7350
-F 0 "#PWR113" H 5500 7100 50  0001 C CNN
+F 0 "#PWR110" H 5500 7100 50  0001 C CNN
 F 1 "GND" H 5500 7200 50  0000 C CNN
 F 2 "" H 5500 7350 50  0000 C CNN
@@
 $EndComp
 $Comp
-L +3V3 #PWR114
+L +3V3 #PWR111
 U 1 1 588947E2
 P 6500 6800
-F 0 "#PWR114" H 6500 6650 50  0001 C CNN
+F 0 "#PWR111" H 6500 6650 50  0001 C CNN
 F 1 "+3V3" H 6500 6940 50  0000 C CNN
 F 2 "" H 6500 6800 50  0000 C CNN
@@
 $EndComp
 $Comp
-L +5V #PWR110
+L +5V #PWR109
 U 1 1 5889504A
 P 3250 6800
-F 0 "#PWR110" H 3250 6650 50  0001 C CNN
+F 0 "#PWR109" H 3250 6650 50  0001 C CNN
 F 1 "+5V" H 3250 6940 50  0000 C CNN
 F 2 "" H 3250 6800 50  0000 C CNN
@@
 $EndComp
 $Comp
-L GND #PWR116
+L GND #PWR113
 U 1 1 5889B140
 P 8950 5800
-F 0 "#PWR116" H 8950 5550 50  0001 C CNN
+F 0 "#PWR113" H 8950 5550 50  0001 C CNN
 F 1 "GND" H 8950 5650 50  0000 C CNN
 F 2 "" H 8950 5800 50  0000 C CNN
@@
 F 3 "" H 1350 2950 50  0000 C CNN
 	1    1350 2950
-	1    0    0    -1
-$EndComp
-$Comp
-L +3V3 #PWR109
-U 1 1 5889DFDA
-P 3000 1950
-F 0 "#PWR109" H 3000 1800 50  0001 C CNN
-F 1 "+3V3" H 3000 2090 50  0000 C CNN
-F 2 "" H 3000 1950 50  0000 C CNN
-F 3 "" H 3000 1950 50  0000 C CNN
-	1    3000 1950
 	1    0    0    -1
 $EndComp
@@
 $EndComp
 $Comp
-L GND #PWR117
+L GND #PWR114
 U 1 1 58F680A4
 P 9700 5350
-F 0 "#PWR117" H 9700 5100 50  0001 C CNN
+F 0 "#PWR114" H 9700 5100 50  0001 C CNN
 F 1 "GND" H 9700 5200 50  0000 C CNN
 F 2 "" H 9700 5350 50  0000 C CNN
@@
 $EndComp
 $Comp
-L GND #PWR118
+L GND #PWR115
 U 1 1 58F6B2FF
 P 9950 5650
-F 0 "#PWR118" H 9950 5400 50  0001 C CNN
+F 0 "#PWR115" H 9950 5400 50  0001 C CNN
 F 1 "GND" H 9950 5500 50  0000 C CNN
 F 2 "" H 9950 5650 50  0000 C CNN
@@
 	0    -1   -1   0
 $EndComp
-$Comp
-L DB9_FEMALE J102
-U 1 1 58F94E12
-P 4100 1800
-F 0 "J102" H 4100 2350 50  0000 C CNN
-F 1 "Probe position sensors" V 4300 1800 50  0000 C CNN
-F 2 "" H 4100 1800 50  0001 C CNN
-F 3 "" H 4100 1800 50  0001 C CNN
-	1    4100 1800
-	-1   0    0    -1
-$EndComp
-$Comp
-L GND #PWR112
-U 1 1 58F97C6C
-P 4600 2200
-F 0 "#PWR112" H 4600 1950 50  0001 C CNN
-F 1 "GND" H 4600 2050 50  0000 C CNN
-F 2 "" H 4600 2200 50  0001 C CNN
-F 3 "" H 4600 2200 50  0001 C CNN
-	1    4600 2200
-	0    -1   -1   0
-$EndComp
-$Comp
-L +5V #PWR111
-U 1 1 58F9B376
-P 4600 1300
-F 0 "#PWR111" H 4600 1150 50  0001 C CNN
-F 1 "+5V" H 4600 1440 50  0000 C CNN
-F 2 "" H 4600 1300 50  0000 C CNN
-F 3 "" H 4600 1300 50  0000 C CNN
-	1    4600 1300
-	1    0    0    -1
-$EndComp
 Wire Wire Line
 	1450 1300 1450 1400
@@
 Connection ~ 4750 6800
 Wire Wire Line
-	1350 1600 3600 1600
-Wire Wire Line
-	1350 1500 3700 1500
-Wire Wire Line
-	5050 2450 3700 2450
-Wire Wire Line
-	3700 2450 3700 1500
-Wire Wire Line
-	3600 1600 3600 2550
-Wire Wire Line
-	3600 2550 5050 2550
+	3050 2450 5050 2450
+Wire Wire Line
+	2950 2550 5050 2550
 Wire Wire Line
 	1850 1700 1750 1700
@@
 Wire Wire Line
 	8950 5800 8850 5800
-Wire Wire Line
-	4400 1500 4950 1500
-Wire Wire Line
-	4950 1500 4950 1600
-Wire Wire Line
-	4950 1600 5050 1600
-Wire Wire Line
-	5050 1700 4850 1700
-Wire Wire Line
-	4850 1700 4850 1600
-Wire Wire Line
-	4850 1600 4400 1600
-Wire Wire Line
-	4400 1700 4750 1700
-Wire Wire Line
-	4750 1700 4750 1800
-Wire Wire Line
-	4750 1800 5050 1800
-Wire Wire Line
-	4400 1900 5050 1900
-Wire Wire Line
-	4400 2000 5050 2000
-Wire Wire Line
-	5050 2100 4400 2100
-Wire Wire Line
-	4400 2200 4600 2200
-Wire Wire Line
-	4400 1400 4500 1400
-Wire Wire Line
-	4500 1400 4500 2200
-Connection ~ 4500 2200
-Wire Wire Line
-	4600 1300 4600 1800
-Wire Wire Line
-	4600 1800 4400 1800
 Text Notes 900  3250 1    60   ~ 0
 Various I2C temperature\nsensors (DS1731)\nBattery, structure, PCBs,\ncupola, camera, ...
@@
 $EndComp
 $Comp
-L GND #PWR115
+L GND #PWR112
 U 1 1 59083068
 P 8750 1000
-F 0 "#PWR115" H 8750 750 50  0001 C CNN
+F 0 "#PWR112" H 8750 750 50  0001 C CNN
 F 1 "GND" H 8750 850 50  0000 C CNN
 F 2 "" H 8750 1000 50  0001 C CNN
@@
 Wire Wire Line
 	4300 4950 5050 4950
+$Sheet
+S 3300 1500 1350 700
+U 591DE5BC
+F0 "Heat_Probe_Encoder" 60
+F1 "heat_probe_encoder.sch" 60
+F2 "ENC1_A" O R 4650 1600 60
+F3 "ENC1_B" O R 4650 1700 60
+F4 "ENC2_A" O R 4650 1800 60
+F5 "ENC2_B" O R 4650 1900 60
+F6 "ENC3_A" O R 4650 2000 60
+F7 "ENC3_B" O R 4650 2100 60
+$EndSheet
+Wire Wire Line
+	1350 1500 3050 1500
+Wire Wire Line
+	3050 1500 3050 2450
+Wire Wire Line
+	2950 2550 2950 1600
+Wire Wire Line
+	2950 1600 1350 1600
+Wire Wire Line
+	4650 2100 5050 2100
+Wire Wire Line
+	5050 2000 4650 2000
+Wire Wire Line
+	4650 1900 5050 1900
+Wire Wire Line
+	5050 1800 4650 1800
+Wire Wire Line
+	4650 1700 5050 1700
+Wire Wire Line
+	5050 1600 4650 1600
 $EndSCHEMATC

Commit message: [mainboard] remove ground loop via camera, docs: update SVGs
Parts:
- added R108: NC, symbol R
Connections:
- net GND: now also R108.2; no longer J103.6
- new net: J103.6, R108.1
Other:
- moved on the sheet: J103
Changed lines of the file:
@@
 Title "Mainboard overview"
 Date "2017-03-14"
-Rev "11"
+Rev "12"
 Comp "VIPER"
 Comment1 ""
@@
 L DB9_FEMALE J103
 U 1 1 59082736
-P 9400 1200
-F 0 "J103" H 9400 1750 50  0000 C CNN
-F 1 "Camera board" V 9600 1200 50  0000 C CNN
-F 2 "" H 9400 1200 50  0001 C CNN
-F 3 "" H 9400 1200 50  0001 C CNN
-	1    9400 1200
+P 9900 1200
+F 0 "J103" H 9900 1750 50  0000 C CNN
+F 1 "Camera board" V 10100 1200 50  0000 C CNN
+F 2 "" H 9900 1200 50  0001 C CNN
+F 3 "" H 9900 1200 50  0001 C CNN
+	1    9900 1200
 	1    0    0    -1
 $EndComp
@@
 	8600 1600 8600 800
 Wire Wire Line
-	8600 800  9100 800
-NoConn ~ 9100 1100
-NoConn ~ 9100 1200
-NoConn ~ 9100 1300
-NoConn ~ 9100 1400
-NoConn ~ 9100 1500
-NoConn ~ 9100 1600
+	8600 800  9600 800
+NoConn ~ 9600 1100
+NoConn ~ 9600 1200
+NoConn ~ 9600 1300
+NoConn ~ 9600 1400
+NoConn ~ 9600 1500
+NoConn ~ 9600 1600
 Wire Wire Line
 	8750 1000 8750 900
 Wire Wire Line
-	8750 900  9100 900
-Wire Wire Line
-	9100 1000 8900 1000
-Wire Wire Line
-	8900 1000 8900 1700
+	9150 900  9600 900
+Wire Wire Line
+	8900 1000 9600 1000
+Wire Wire Line
+	8900 1700 8900 1000
 $Comp
 L DB37_MALE J101
@@
 Wire Wire Line
 	5050 1600 4650 1600
+$Comp
+L R R108
+U 1 1 59204DCC
+P 9000 900
+F 0 "R108" V 9080 900 50  0000 C CNN
+F 1 "NC" V 9000 900 50  0000 C CNN
+F 2 "" V 8930 900 50  0001 C CNN
+F 3 "" H 9000 900 50  0001 C CNN
+	1    9000 900
+	0    1    1    0
+$EndComp
+Wire Wire Line
+	8750 900  8850 900
 $EndSCHEMATC

Commit message: [mainboard] update board-to-board connector to powerboard; docs: update SVGs
Parts:
- removed J101: Powerboard <-> Mainboard, symbol DB37_MALE
- added J101: Powerboard <-> Mainboard, symbol CONN_01X40
Connections:
- net +5V: now also J101.2 (P2), J101.3 (P3)
- net Boost24V_EN: now also J101.26 (P26)
- net Brake_EN: now also J101.4 (P4)
- net Cam_Light_EN: now also J101.23 (P23)
- net Charge_EN: now also J101.21 (P21)
- net Charge_status: now also J101.22 (P22)
- net Encoder_A+: now also J101.28 (P28)
- net Encoder_B+: now also J101.29 (P29)
- net GND: now also J101.1 (P1), J101.11 (P11), J101.15 (P15), J101.20 (P20), J101.24 (P24), J101.27 (P27), J101.30 (P30), J101.34 (P34), J101.40 (P40)
- net Hall_U: now also J101.31 (P31)
- net Hall_V: now also J101.32 (P32)
- net Hall_W: now also J101.33 (P33)
- net LO: now also J101.35 (P35)
- net Lens_Heat_EN: now also J101.25 (P25)
- net Motor_U_N: now also J101.6 (P6)
- net Motor_U_P: now also J101.5 (P5)
- net Motor_V_N: now also J101.8 (P8)
- net Motor_V_P: now also J101.7 (P7)
- net Motor_W_N: now also J101.10 (P10)
- net Motor_W_P: now also J101.9 (P9)
- net Probe1_EN: now also J101.12 (P12)
- net Probe2_EN: now also J101.13 (P13)
- net Probe3_EN: now also J101.14 (P14)
- net RX: now also J101.39 (P39)
- net SODS: now also J101.37 (P37)
- net SOE: now also J101.36 (P36)
- net TX: now also J101.38 (P38)
- net extADC_SPI_CS1: now also J101.19 (P19)
- net extADC_SPI_MISO: now also J101.17 (P17)
- net extADC_SPI_MOSI: now also J101.18 (P18)
- net extADC_SPI_SCK: now also J101.16 (P16)
Changed lines of the file:
@@
 Wire Wire Line
 	8900 1700 8900 1000
-$Comp
-L DB37_MALE J101
-U 1 1 5908B98D
-P 800 5500
-F 0 "J101" H 800 7500 50  0000 C CNN
-F 1 "Powerboard <-> Mainboard" V 1000 5500 50  0000 C CNN
-F 2 "" H 800 5500 50  0001 C CNN
-F 3 "" H 800 5500 50  0001 C CNN
-	1    800  5500
-	-1   0    0    1
-$EndComp
-Text Label 1950 5900 2    60   ~ 0
+Text Label 1950 6100 2    60   ~ 0
 Lens_Heat_EN
 Text Label 1950 5000 2    60   ~ 0
@@
 Text Label 1950 4800 2    60   ~ 0
 Probe1_EN
+Text Label 1950 5900 2    60   ~ 0
+Cam_Light_EN
 Text Label 1950 5800 2    60   ~ 0
-Cam_Light_EN
+Charge_status
+Text Label 1950 6200 2    60   ~ 0
+Boost24V_EN
 Text Label 1950 5700 2    60   ~ 0
-Charge_status
-Text Label 1950 6000 2    60   ~ 0
-Boost24V_EN
-Text Label 1950 5600 2    60   ~ 0
 Charge_EN
+Text Label 1950 6700 2    60   ~ 0
+Hall_U
+Text Label 1950 6800 2    60   ~ 0
+Hall_V
+Text Label 1950 6900 2    60   ~ 0
+Hall_W
+Text Label 1950 6400 2    60   ~ 0
+Encoder_A+
 Text Label 1950 6500 2    60   ~ 0
-Hall_U
-Text Label 1950 6600 2    60   ~ 0
-Hall_V
-Text Label 1950 6700 2    60   ~ 0
-Hall_W
-Text Label 1950 6200 2    60   ~ 0
-Encoder_A+
-Text Label 1950 6300 2    60   ~ 0
 Encoder_B+
-Text Label 1950 6800 2    60   ~ 0
+Text Label 1950 7100 2    60   ~ 0
 LO
-Text Label 1950 6900 2    60   ~ 0
+Text Label 1950 7200 2    60   ~ 0
 SOE
-Text Label 1950 7000 2    60   ~ 0
+Text Label 1950 7300 2    60   ~ 0
 SODS
-Text Label 1950 7100 2    60   ~ 0
+Text Label 1950 7400 2    60   ~ 0
 TX
-Text Label 1950 7200 2    60   ~ 0
+Text Label 1950 7500 2    60   ~ 0
 RX
 $Comp
 L GND #PWR101
 U 1 1 5913059A
-P 1200 7400
-F 0 "#PWR101" H 1200 7150 50  0001 C CNN
-F 1 "GND" H 1200 7250 50  0000 C CNN
-F 2 "" H 1200 7400 50  0001 C CNN
-F 3 "" H 1200 7400 50  0001 C CNN
-	1    1200 7400
-	1    0    0    -1
+P 1300 7700
+F 0 "#PWR101" H 1300 7450 50  0001 C CNN
+F 1 "GND" H 1300 7550 50  0000 C CNN
+F 2 "" H 1300 7700 50  0001 C CNN
+F 3 "" H 1300 7700 50  0001 C CNN
+	1    1300 7700
+	0    -1   -1   0
 $EndComp
 $Comp
@@
 Brake_EN
 Wire Wire Line
-	1200 3700 1200 7400
-Wire Wire Line
-	1200 7300 1100 7300
+	1200 7600 1100 7600
 Wire Wire Line
 	1200 3700 1100 3700
-Connection ~ 1200 7300
-Wire Wire Line
-	1100 6400 1200 6400
-Connection ~ 1200 6400
-Wire Wire Line
-	1100 5500 1200 5500
-Connection ~ 1200 5500
+Connection ~ 1200 7600
+Wire Wire Line
+	1200 6600 1100 6600
+Connection ~ 1200 6600
+Wire Wire Line
+	1200 5600 1100 5600
+Connection ~ 1200 5600
 Wire Wire Line
 	1400 3600 1400 3900
@@
 Connection ~ 1400 3800
 Wire Wire Line
-	1950 7200 1100 7200
-Wire Wire Line
-	1100 7100 1950 7100
-Wire Wire Line
-	1950 7000 1100 7000
+	1950 7500 1100 7500
+Wire Wire Line
+	1100 7400 1950 7400
+Wire Wire Line
+	1950 7300 1100 7300
+Wire Wire Line
+	1100 7200 1950 7200
+Wire Wire Line
+	1950 7100 1100 7100
 Wire Wire Line
 	1100 6900 1950 6900
@@
 	1100 6700 1950 6700
 Wire Wire Line
-	1950 6600 1100 6600
-Wire Wire Line
 	1100 6500 1950 6500
 Wire Wire Line
-	1100 6300 1950 6300
-Wire Wire Line
-	1950 6200 1100 6200
-Wire Wire Line
-	1100 5900 1950 5900
-Wire Wire Line
-	1950 5800 1100 5800
-Wire Wire Line
-	1100 5700 1950 5700
-Wire Wire Line
-	1950 5600 1100 5600
-Wire Wire Line
-	1100 5400 1950 5400
-Wire Wire Line
-	1950 5300 1100 5300
-Wire Wire Line
-	1100 5200 1950 5200
-Wire Wire Line
-	1950 5100 1100 5100
+	1950 6400 1100 6400
+Wire Wire Line
+	1100 6100 1950 6100
+Wire Wire Line
+	1950 5900 1100 5900
+Wire Wire Line
+	1100 5800 1950 5800
+Wire Wire Line
+	1950 5700 1100 5700
+Wire Wire Line
+	1100 5500 1950 5500
+Wire Wire Line
+	1950 5400 1100 5400
+Wire Wire Line
+	1100 5300 1950 5300
+Wire Wire Line
+	1950 5200 1100 5200
 Wire Wire Line
 	1100 5000 1950 5000
@@
 	1100 4000 1950 4000
 Wire Wire Line
-	1100 6100 1200 6100
-Connection ~ 1200 6100
-Wire Wire Line
-	1100 6000 1950 6000
+	1200 6300 1100 6300
+Connection ~ 1200 6300
+Wire Wire Line
+	1100 6200 1950 6200
 Wire Wire Line
 	1100 4700 1200 4700
@@
 Wire Wire Line
 	4300 3550 5050 3550
-Text Label 1950 5100 2    60   ~ 0
+Text Label 1950 5200 2    60   ~ 0
 extADC_SPI_SCK
-Text Label 1950 5200 2    60   ~ 0
+Text Label 1950 5300 2    60   ~ 0
 extADC_SPI_MISO
-Text Label 1950 5300 2    60   ~ 0
+Text Label 1950 5400 2    60   ~ 0
 extADC_SPI_MOSI
-Text Label 1950 5400 2    60   ~ 0
+Text Label 1950 5500 2    60   ~ 0
 extADC_SPI_CS1
 Text Label 4300 3850 0    60   ~ 0
@@
 Wire Wire Line
 	8750 900  8850 900
+$Comp
+L CONN_01X40 J101
+U 1 1 592203A3
+P 900 5650
+F 0 "J101" H 900 7700 50  0000 C CNN
+F 1 "Powerboard <-> Mainboard" V 1000 5650 50  0000 C CNN
+F 2 "" H 900 5650 50  0001 C CNN
+F 3 "" H 900 5650 50  0001 C CNN
+	1    900  5650
+	-1   0    0    -1
+$EndComp
+Wire Wire Line
+	1200 3700 1200 7700
+Wire Wire Line
+	1200 5100 1100 5100
+Connection ~ 1200 5100
+Wire Wire Line
+	1200 6000 1100 6000
+Connection ~ 1200 6000
+Wire Wire Line
+	1200 7000 1100 7000
+Connection ~ 1200 7000
+Wire Wire Line
+	1200 7700 1300 7700
 $EndSCHEMATC

Commit message: [mainboard] update connectors, select most footprints; docs: update SVGs
Parts:
- removed P101: Temperature, symbol CONN_01X04
- removed P102: Pressure, symbol CONN_01X04
- added J?: Temperature & Pressure, symbol DB9_FEMALE
- C104, C105, D101, D102, D103: footprint (none) -> Capacitors_SMD:C_0603
- J101: footprint (none) -> Pin_Headers:Pin_Header_Straight_2x20_Pitch2.54mm
- R101, R102, R103, R104, R105, R106, R107, R108: footprint (none) -> Resistors_SMD:R_0603
Connections:
- net +3V3: now also J?.7, J?.8
- net GND: now also J?.1, J?.3, J?.5
- net pressure_SCL: now also J?.6
- net pressure_SDA: now also J?.2
- net temperature_SCL: now also J?.4
- net temperature_SDA: now also J?.9
Other:
- note added: "Pressure sensor:\nAMSYS 5915-0010-D (3.3V)\nor First Sensor HCLA"
- note removed: "AMSYS\n5915-0010-D\n(3.3V)\nor First Sensor HCLA"

Commit message: [mainboard] layout: footprints assigned, first placement
Parts:
- J102: renamed from J?; footprint (none) -> Connectors:DB9FD
- J103: footprint (none) -> Connectors:DB9FD
- SW101, SW102: footprint (none) -> Buttons_Switches_SMD:SW_SPST_FSMSM
Changed lines of the file:
@@
 $EndComp
 $Comp
-L GND #PWR03
+L GND #PWR01
 U 1 1 588947DC
 P 5500 7350
-F 0 "#PWR03" H 5500 7100 50  0001 C CNN
+F 0 "#PWR01" H 5500 7100 50  0001 C CNN
 F 1 "GND" H 5500 7200 50  0000 C CNN
 F 2 "" H 5500 7350 50  0000 C CNN
@@
 $EndComp
 $Comp
-L +3V3 #PWR04
+L +3V3 #PWR02
 U 1 1 588947E2
 P 6500 6800
-F 0 "#PWR04" H 6500 6650 50  0001 C CNN
+F 0 "#PWR02" H 6500 6650 50  0001 C CNN
 F 1 "+3V3" H 6500 6940 50  0000 C CNN
 F 2 "" H 6500 6800 50  0000 C CNN
@@
 $EndComp
 $Comp
-L +5V #PWR05
+L +5V #PWR03
 U 1 1 5889504A
 P 3250 6800
-F 0 "#PWR05" H 3250 6650 50  0001 C CNN
+F 0 "#PWR03" H 3250 6650 50  0001 C CNN
 F 1 "+5V" H 3250 6940 50  0000 C CNN
 F 2 "" H 3250 6800 50  0000 C CNN
@@
 $EndComp
 $Comp
-L GND #PWR06
+L GND #PWR04
 U 1 1 5889B140
 P 8950 5800
-F 0 "#PWR06" H 8950 5550 50  0001 C CNN
+F 0 "#PWR04" H 8950 5550 50  0001 C CNN
 F 1 "GND" H 8950 5650 50  0000 C CNN
 F 2 "" H 8950 5800 50  0000 C CNN
@@
 $EndComp
 $Comp
-L +3V3 #PWR07
+L +3V3 #PWR05
 U 1 1 5889CCC2
 P 1300 2150
-F 0 "#PWR07" H 1300 2000 50  0001 C CNN
+F 0 "#PWR05" H 1300 2000 50  0001 C CNN
 F 1 "+3V3" H 1300 2290 50  0000 C CNN
 F 2 "" H 1300 2150 50  0000 C CNN
@@
 $EndComp
 $Comp
-L GND #PWR08
+L GND #PWR06
 U 1 1 5889CF45
 P 1100 2650
-F 0 "#PWR08" H 1100 2400 50  0001 C CNN
+F 0 "#PWR06" H 1100 2400 50  0001 C CNN
 F 1 "GND" H 1100 2500 50  0000 C CNN
 F 2 "" H 1100 2650 50  0000 C CNN
@@
 $EndComp
 $Comp
-L +3V3 #PWR09
+L +3V3 #PWR07
 U 1 1 58C90F6C
 P 2500 1700
-F 0 "#PWR09" H 2500 1550 50  0001 C CNN
+F 0 "#PWR07" H 2500 1550 50  0001 C CNN
 F 1 "+3V3" H 2500 1840 50  0000 C CNN
 F 2 "" H 2500 1700 50  0000 C CNN
@@
 $EndComp
 $Comp
-L +3V3 #PWR010
+L +3V3 #PWR08
 U 1 1 58F52861
 P 2400 2850
-F 0 "#PWR010" H 2400 2700 50  0001 C CNN
+F 0 "#PWR08" H 2400 2700 50  0001 C CNN
 F 1 "+3V3" H 2400 2990 50  0000 C CNN
 F 2 "" H 2400 2850 50  0000 C CNN
@@
 F 0 "SW101" H 8700 5910 50  0000 C CNN
 F 1 "SW_PUSH" H 8550 5720 50  0000 C CNN
-F 2 "" H 8550 5800 50  0001 C CNN
+F 2 "Buttons_Switches_SMD:SW_SPST_FSMSM" H 8550 5800 50  0001 C CNN
 F 3 "" H 8550 5800 50  0000 C CNN
 	1    8550 5800
@@
 F 0 "SW102" H 9700 5760 50  0000 C CNN
 F 1 "SW_PUSH" H 9550 5570 50  0000 C CNN
-F 2 "" H 9550 5650 50  0001 C CNN
+F 2 "Buttons_Switches_SMD:SW_SPST_FSMSM" H 9550 5650 50  0001 C CNN
 F 3 "" H 9550 5650 50  0000 C CNN
 	1    9550 5650
@@
 $EndComp
 $Comp
-L GND #PWR011
+L GND #PWR09
 U 1 1 58F680A4
 P 9700 5350
-F 0 "#PWR011" H 9700 5100 50  0001 C CNN
+F 0 "#PWR09" H 9700 5100 50  0001 C CNN
 F 1 "GND" H 9700 5200 50  0000 C CNN
 F 2 "" H 9700 5350 50  0000 C CNN
@@
 $EndComp
 $Comp
-L GND #PWR012
+L GND #PWR010
 U 1 1 58F6B2FF
 P 9950 5650
-F 0 "#PWR012" H 9950 5400 50  0001 C CNN
+F 0 "#PWR010" H 9950 5400 50  0001 C CNN
 F 1 "GND" H 9950 5500 50  0000 C CNN
 F 2 "" H 9950 5650 50  0000 C CNN
@@
 F 0 "J103" H 9900 1750 50  0000 C CNN
 F 1 "Camera board" V 10100 1200 50  0000 C CNN
-F 2 "" H 9900 1200 50  0001 C CNN
+F 2 "Connectors:DB9FD" H 9900 1200 50  0001 C CNN
 F 3 "" H 9900 1200 50  0001 C CNN
 	1    9900 1200
@@
 $EndComp
 $Comp
-L GND #PWR013
+L GND #PWR011
 U 1 1 59083068
 P 8750 1000
-F 0 "#PWR013" H 8750 750 50  0001 C CNN
+F 0 "#PWR011" H 8750 750 50  0001 C CNN
 F 1 "GND" H 8750 850 50  0000 C CNN
 F 2 "" H 8750 1000 50  0001 C CNN
@@
 RX
 $Comp
-L GND #PWR014
+L GND #PWR012
 U 1 1 5913059A
 P 1300 7700
-F 0 "#PWR014" H 1300 7450 50  0001 C CNN
+F 0 "#PWR012" H 1300 7450 50  0001 C CNN
 F 1 "GND" H 1300 7550 50  0000 C CNN
 F 2 "" H 1300 7700 50  0001 C CNN
@@
 $EndComp
 $Comp
-L +5V #PWR015
+L +5V #PWR013
 U 1 1 591305A0
 P 1400 3600
-F 0 "#PWR015" H 1400 3450 50  0001 C CNN
+F 0 "#PWR013" H 1400 3450 50  0001 C CNN
 F 1 "+5V" H 1400 3740 50  0000 C CNN
 F 2 "" H 1400 3600 50  0000 C CNN
@@
 	1200 7700 1300 7700
 $Comp
-L DB9_FEMALE J?
+L DB9_FEMALE J102
 U 1 1 59285E82
 P 700 2150
-F 0 "J?" H 700 2700 50  0000 C CNN
+F 0 "J102" H 700 2700 50  0000 C CNN
 F 1 "Temperature & Pressure" H 400 1350 50  0000 C CNN
-F 2 "" H 700 2150 50  0001 C CNN
+F 2 "Connectors:DB9FD" H 700 2150 50  0001 C CNN
 F 3 "" H 700 2150 50  0001 C CNN
 	1    700  2150

Commit message: [mainboard] add more local net labels, add not-connected flags
Connections:
- net 5V_filtered: now reaches C102.1, C103.1, C104.1, L101.2, U101.3 (VI)
- net LED3_R: now reaches D102.2 (A), R106.1
- net LED1_R: now reaches D101.2 (A), R105.1
- net LED2_R: now reaches D103.2 (A), R107.1
- net CAM_GND: now reaches J103.6, R108.1
Changed lines of the file:
@@
 Wire Wire Line
 	1350 2750 5050 2750
+Text Label 8400 5250 0    20   ~ 0
+LED1_R
+Text Label 8900 5350 0    20   ~ 0
+LED2_R
+Text Label 8400 5450 0    20   ~ 0
+LED3_R
+Text Label 4450 6800 0    60   ~ 0
+5V_filtered
+Text Label 9200 900  0    60   ~ 0
+CAM_GND
 $EndSCHEMATC

Commit message: [mainboard] layout: footprint placement
Parts:
- D101, D102, D103: footprint Capacitors_SMD:C_0603 -> LEDs:LED_0603
Changed lines of the file:
@@
 F 0 "D101" H 9100 5300 50  0000 C CNN
 F 1 "RED" H 8950 5150 50  0000 C CNN
-F 2 "Capacitors_SMD:C_0603" H 8950 5250 50  0001 C CNN
+F 2 "LEDs:LED_0603" H 8950 5250 50  0001 C CNN
 F 3 "" H 8950 5250 50  0001 C CNN
 	1    8950 5250
@@
 F 0 "D102" H 8850 5500 50  0000 C CNN
 F 1 "BLUE" H 8950 5550 50  0000 C CNN
-F 2 "Capacitors_SMD:C_0603" H 8950 5450 50  0001 C CNN
+F 2 "LEDs:LED_0603" H 8950 5450 50  0001 C CNN
 F 3 "" H 8950 5450 50  0001 C CNN
 	1    8950 5450
@@
 F 0 "D103" H 9250 5400 50  0000 C CNN
 F 1 "GREEN" H 9350 5200 50  0000 C CNN
-F 2 "Capacitors_SMD:C_0603" H 9350 5350 50  0001 C CNN
+F 2 "LEDs:LED_0603" H 9350 5350 50  0001 C CNN
 F 3 "" H 9350 5350 50  0001 C CNN
 	1    9350 5350
