File: boards/mainboard/heat_probe_encoder.sch (KiCad schematic (older format))
At the start: 33 parts, among them J1201 ENC1_A, J1202 ENC1_B, J1203 ENC2_A, J1204 ENC2_B, J1205 ENC3_A, J1206 ENC3_B, U1201 Heat probe encoder, U1202 DS26LV32AT, U1203 DS26LV32AT

Commit message: [mainboard] component placement (wip...)
Parts:
- added C1207, C1208: 100n, Capacitors_SMD:C_0603, symbol C
Connections:
- net +3V3: now also C1207.1, C1208.1
- net GND: now also C1207.2, C1208.2
Changed lines of the file:
@@
 $EndComp
 $Comp
-L GND #PWR1212
+L GND #PWR1216
 U 1 1 591E1E04
 P 8300 4050
-F 0 "#PWR1212" H 8300 3800 50  0001 C CNN
+F 0 "#PWR1216" H 8300 3800 50  0001 C CNN
 F 1 "GND" H 8300 3900 50  0000 C CNN
 F 2 "" H 8300 4050 50  0001 C CNN
@@
 $EndComp
 $Comp
-L +3V3 #PWR1211
+L +3V3 #PWR1215
 U 1 1 591E2628
 P 6900 1700
-F 0 "#PWR1211" H 6900 1550 50  0001 C CNN
+F 0 "#PWR1215" H 6900 1550 50  0001 C CNN
 F 1 "+3V3" H 6900 1840 50  0000 C CNN
 F 2 "" H 6900 1700 50  0001 C CNN
@@
 	1    0    0    -1
 $EndComp
+$Comp
+L C C1207
+U 1 1 591CB88F
+P 6450 5950
+F 0 "C1207" H 6475 6050 50  0000 L CNN
+F 1 "100n" H 6475 5850 50  0000 L CNN
+F 2 "Capacitors_SMD:C_0603" H 6488 5800 50  0001 C CNN
+F 3 "" H 6450 5950 50  0001 C CNN
+	1    6450 5950
+	1    0    0    -1
+$EndComp
+$Comp
+L +3V3 #PWR1211
+U 1 1 591CB9CB
+P 6450 5700
+F 0 "#PWR1211" H 6450 5550 50  0001 C CNN
+F 1 "+3V3" H 6450 5840 50  0000 C CNN
+F 2 "" H 6450 5700 50  0001 C CNN
+F 3 "" H 6450 5700 50  0001 C CNN
+	1    6450 5700
+	1    0    0    -1
+$EndComp
+$Comp
+L GND #PWR1212
+U 1 1 591CBA3C
+P 6450 6200
+F 0 "#PWR1212" H 6450 5950 50  0001 C CNN
+F 1 "GND" H 6450 6050 50  0000 C CNN
+F 2 "" H 6450 6200 50  0001 C CNN
+F 3 "" H 6450 6200 50  0001 C CNN
+	1    6450 6200
+	1    0    0    -1
+$EndComp
+Wire Wire Line
+	6450 6200 6450 6100
+Wire Wire Line
+	6450 5800 6450 5700
+$Comp
+L C C1208
+U 1 1 591CC192
+P 6850 4500
+F 0 "C1208" H 6875 4600 50  0000 L CNN
+F 1 "100n" H 6875 4400 50  0000 L CNN
+F 2 "Capacitors_SMD:C_0603" H 6888 4350 50  0001 C CNN
+F 3 "" H 6850 4500 50  0001 C CNN
+	1    6850 4500
+	1    0    0    -1
+$EndComp
+$Comp
+L +3V3 #PWR1213
+U 1 1 591CC198
+P 6850 4250
+F 0 "#PWR1213" H 6850 4100 50  0001 C CNN
+F 1 "+3V3" H 6850 4390 50  0000 C CNN
+F 2 "" H 6850 4250 50  0001 C CNN
+F 3 "" H 6850 4250 50  0001 C CNN
+	1    6850 4250
+	1    0    0    -1
+$EndComp
+$Comp
+L GND #PWR1214
+U 1 1 591CC19E
+P 6850 4750
+F 0 "#PWR1214" H 6850 4500 50  0001 C CNN
+F 1 "GND" H 6850 4600 50  0000 C CNN
+F 2 "" H 6850 4750 50  0001 C CNN
+F 3 "" H 6850 4750 50  0001 C CNN
+	1    6850 4750
+	1    0    0    -1
+$EndComp
+Wire Wire Line
+	6850 4750 6850 4650
+Wire Wire Line
+	6850 4350 6850 4250
 $EndSCHEMATC
