File: boards/mainboard/mainboard-LTC2984_2.sch (KiCad schematic (older format))
At the start: 33 parts, among them U301 LTC2984

Commit message: [mainboard] layout: footprints assigned, first placement
Parts:
- R302: footprint Resistors_ThroughHole:Resistor_Horizontal_RM7mm -> Resistors_THT:R_Axial_DIN0204_L3.6mm_D1.6mm_P5.08mm_Horizontal
Changed lines of the file:
@@
 F 0 "R302" V 4350 2200 50  0000 C CNN
 F 1 "2k00" V 4450 2200 50  0000 C CNN
-F 2 "Resistors_ThroughHole:Resistor_Horizontal_RM7mm" V 4380 2200 50  0001 C CNN
+F 2 "Resistors_THT:R_Axial_DIN0204_L3.6mm_D1.6mm_P5.08mm_Horizontal" V 4380 2200 50  0001 C CNN
 F 3 "" H 4450 2200 50  0000 C CNN
 	1    4450 2200
@@
 $EndComp
 $Comp
-L GND #PWR017
+L GND #PWR015
 U 1 1 58FFF542
 P 5650 1600
-F 0 "#PWR017" H 5650 1350 50  0001 C CNN
+F 0 "#PWR015" H 5650 1350 50  0001 C CNN
 F 1 "GND" H 5650 1450 50  0000 C CNN
 F 2 "" H 5650 1600 50  0000 C CNN
@@
 $EndComp
 $Comp
-L GND #PWR018
+L GND #PWR016
 U 1 1 587B30AA
 P 5650 4850
-F 0 "#PWR018" H 5650 4600 50  0001 C CNN
+F 0 "#PWR016" H 5650 4600 50  0001 C CNN
 F 1 "GND" H 5650 4700 50  0000 C CNN
 F 2 "" H 5650 4850 50  0000 C CNN
@@
 $EndComp
 $Comp
-L GND #PWR019
+L GND #PWR017
 U 1 1 58FFF582
 P 8200 1750
-F 0 "#PWR019" H 8200 1500 50  0001 C CNN
+F 0 "#PWR017" H 8200 1500 50  0001 C CNN
 F 1 "GND" H 8200 1600 50  0000 C CNN
 F 2 "" H 8200 1750 50  0000 C CNN
@@
 $EndComp
 $Comp
-L GND #PWR020
+L GND #PWR018
 U 1 1 58FFF58D
 P 7000 1150
-F 0 "#PWR020" H 7000 900 50  0001 C CNN
+F 0 "#PWR018" H 7000 900 50  0001 C CNN
 F 1 "GND" H 7000 1000 50  0000 C CNN
 F 2 "" H 7000 1150 50  0000 C CNN
@@
 $EndComp
 $Comp
-L GND #PWR021
+L GND #PWR019
 U 1 1 58FFF59B
 P 7100 5050
-F 0 "#PWR021" H 7100 4800 50  0001 C CNN
+F 0 "#PWR019" H 7100 4800 50  0001 C CNN
 F 1 "GND" H 7100 4900 50  0000 C CNN
 F 2 "" H 7100 5050 50  0000 C CNN
@@
 $EndComp
 $Comp
-L GND #PWR022
+L GND #PWR020
 U 1 1 58FFF5AD
 P 7300 6150
-F 0 "#PWR022" H 7300 5900 50  0001 C CNN
+F 0 "#PWR020" H 7300 5900 50  0001 C CNN
 F 1 "GND" H 7300 6000 50  0000 C CNN
 F 2 "" H 7300 6150 50  0000 C CNN
@@
 $EndComp
 $Comp
-L GND #PWR023
+L GND #PWR021
 U 1 1 58FFF5B7
 P 7250 1250
-F 0 "#PWR023" H 7250 1000 50  0001 C CNN
+F 0 "#PWR021" H 7250 1000 50  0001 C CNN
 F 1 "GND" H 7250 1100 50  0000 C CNN
 F 2 "" H 7250 1250 50  0000 C CNN
@@
 $EndComp
 $Comp
-L GND #PWR024
+L GND #PWR022
 U 1 1 58FFF5C1
 P 7650 1050
-F 0 "#PWR024" H 7650 800 50  0001 C CNN
+F 0 "#PWR022" H 7650 800 50  0001 C CNN
 F 1 "GND" H 7650 900 50  0000 C CNN
 F 2 "" H 7650 1050 50  0000 C CNN
@@
 $EndComp
 $Comp
-L GND #PWR025
+L GND #PWR023
 U 1 1 58FFF5C4
 P 6550 4600
-F 0 "#PWR025" H 6550 4350 50  0001 C CNN
+F 0 "#PWR023" H 6550 4350 50  0001 C CNN
 F 1 "GND" H 6550 4450 50  0000 C CNN
 F 2 "" H 6550 4600 50  0000 C CNN
@@
 VREF_BYP
 $Comp
-L +3V3 #PWR026
+L +3V3 #PWR024
 U 1 1 587CA05F
 P 7500 5050
-F 0 "#PWR026" H 7500 4900 50  0001 C CNN
+F 0 "#PWR024" H 7500 4900 50  0001 C CNN
 F 1 "+3V3" H 7500 5190 50  0000 C CNN
 F 2 "" H 7500 5050 50  0000 C CNN
@@
 $EndComp
 $Comp
-L +3V3 #PWR027
+L +3V3 #PWR025
 U 1 1 58FFF5D0
 P 7300 5450
-F 0 "#PWR027" H 7300 5300 50  0001 C CNN
+F 0 "#PWR025" H 7300 5300 50  0001 C CNN
 F 1 "+3V3" H 7300 5590 50  0000 C CNN
 F 2 "" H 7300 5450 50  0000 C CNN
@@
 	4300 2000 4250 2000
 $Comp
-L +3V3 #PWR028
+L +3V3 #PWR026
 U 1 1 58FFF5DA
 P 9050 3400
-F 0 "#PWR028" H 9050 3250 50  0001 C CNN
+F 0 "#PWR026" H 9050 3250 50  0001 C CNN
 F 1 "+3V3" H 9050 3540 50  0000 C CNN
 F 2 "" H 9050 3400 50  0000 C CNN
@@
 $EndComp
 $Comp
-L +3V3 #PWR029
+L +3V3 #PWR027
 U 1 1 58FFF5EB
 P 8550 1900
-F 0 "#PWR029" H 8550 1750 50  0001 C CNN
+F 0 "#PWR027" H 8550 1750 50  0001 C CNN
 F 1 "+3V3" H 8550 2040 50  0000 C CNN
 F 2 "" H 8550 1900 50  0000 C CNN

Commit message: [mainboard] first traces routed, some pins in schematic swapped
Parts:
- removed R302: 2k00, Resistors_THT:R_Axial_DIN0204_L3.6mm_D1.6mm_P5.08mm_Horizontal, symbol R
Changed lines of the file:
@@
-$EndComp
-$Comp
-L R R302
-U 1 1 58FFF513
-P 4450 2200
-F 0 "R302" V 4350 2200 50  0000 C CNN
-F 1 "2k00" V 4450 2200 50  0000 C CNN
-F 2 "Resistors_THT:R_Axial_DIN0204_L3.6mm_D1.6mm_P5.08mm_Horizontal" V 4380 2200 50  0001 C CNN
-F 3 "" H 4450 2200 50  0000 C CNN
-	1    4450 2200
-	0    1    1    0
 $EndComp
 $Comp
@@
 Wire Wire Line
 	9050 3400 8950 3400
-Wire Wire Line
-	4250 2200 4300 2200
 Text HLabel 4200 2400 0    60   Input ~ 0
 RTD1_B
