File: boards/mainboard/mainboard-LTC2984_3.sch (KiCad schematic (older format))
At the start: 33 parts, among them U501 LTC2984

Commit message: [mainboard] layout: footprints assigned, first placement
Parts:
- R502: footprint Resistors_ThroughHole:Resistor_Horizontal_RM7mm -> Resistors_THT:R_Axial_DIN0204_L3.6mm_D1.6mm_P5.08mm_Horizontal
Changed lines of the file:
@@
 F 0 "R502" V 4350 2200 50  0000 C CNN
 F 1 "2k00" V 4450 2200 50  0000 C CNN
-F 2 "Resistors_ThroughHole:Resistor_Horizontal_RM7mm" V 4380 2200 50  0001 C CNN
+F 2 "Resistors_THT:R_Axial_DIN0204_L3.6mm_D1.6mm_P5.08mm_Horizontal" V 4380 2200 50  0001 C CNN
 F 3 "" H 4450 2200 50  0000 C CNN
 	1    4450 2200
@@
 $EndComp
 $Comp
-L GND #PWR043
+L GND #PWR041
 U 1 1 58FFF545
 P 5650 1600
-F 0 "#PWR043" H 5650 1350 50  0001 C CNN
+F 0 "#PWR041" H 5650 1350 50  0001 C CNN
 F 1 "GND" H 5650 1450 50  0000 C CNN
 F 2 "" H 5650 1600 50  0000 C CNN
@@
 $EndComp
 $Comp
-L GND #PWR044
+L GND #PWR042
 U 1 1 58FFF580
 P 5650 4850
-F 0 "#PWR044" H 5650 4600 50  0001 C CNN
+F 0 "#PWR042" H 5650 4600 50  0001 C CNN
 F 1 "GND" H 5650 4700 50  0000 C CNN
 F 2 "" H 5650 4850 50  0000 C CNN
@@
 $EndComp
 $Comp
-L GND #PWR045
+L GND #PWR043
 U 1 1 58FFF583
 P 8200 1750
-F 0 "#PWR045" H 8200 1500 50  0001 C CNN
+F 0 "#PWR043" H 8200 1500 50  0001 C CNN
 F 1 "GND" H 8200 1600 50  0000 C CNN
 F 2 "" H 8200 1750 50  0000 C CNN
@@
 $EndComp
 $Comp
-L GND #PWR046
+L GND #PWR044
 U 1 1 58FFF58E
 P 7000 1150
-F 0 "#PWR046" H 7000 900 50  0001 C CNN
+F 0 "#PWR044" H 7000 900 50  0001 C CNN
 F 1 "GND" H 7000 1000 50  0000 C CNN
 F 2 "" H 7000 1150 50  0000 C CNN
@@
 $EndComp
 $Comp
-L GND #PWR047
+L GND #PWR045
 U 1 1 58FFF59F
 P 7100 5050
-F 0 "#PWR047" H 7100 4800 50  0001 C CNN
+F 0 "#PWR045" H 7100 4800 50  0001 C CNN
 F 1 "GND" H 7100 4900 50  0000 C CNN
 F 2 "" H 7100 5050 50  0000 C CNN
@@
 $EndComp
 $Comp
-L GND #PWR048
+L GND #PWR046
 U 1 1 58FFF5AA
 P 7300 6150
-F 0 "#PWR048" H 7300 5900 50  0001 C CNN
+F 0 "#PWR046" H 7300 5900 50  0001 C CNN
 F 1 "GND" H 7300 6000 50  0000 C CNN
 F 2 "" H 7300 6150 50  0000 C CNN
@@
 $EndComp
 $Comp
-L GND #PWR049
+L GND #PWR047
 U 1 1 58FFF5B8
 P 7250 1250
-F 0 "#PWR049" H 7250 1000 50  0001 C CNN
+F 0 "#PWR047" H 7250 1000 50  0001 C CNN
 F 1 "GND" H 7250 1100 50  0000 C CNN
 F 2 "" H 7250 1250 50  0000 C CNN
@@
 $EndComp
 $Comp
-L GND #PWR050
+L GND #PWR048
 U 1 1 58FFF5C0
 P 7650 1050
-F 0 "#PWR050" H 7650 800 50  0001 C CNN
+F 0 "#PWR048" H 7650 800 50  0001 C CNN
 F 1 "GND" H 7650 900 50  0000 C CNN
 F 2 "" H 7650 1050 50  0000 C CNN
@@
 $EndComp
 $Comp
-L GND #PWR051
+L GND #PWR049
 U 1 1 58FFF5C3
 P 6550 4600
-F 0 "#PWR051" H 6550 4350 50  0001 C CNN
+F 0 "#PWR049" H 6550 4350 50  0001 C CNN
 F 1 "GND" H 6550 4450 50  0000 C CNN
 F 2 "" H 6550 4600 50  0000 C CNN
@@
 VREF_BYP
 $Comp
-L +3V3 #PWR052
+L +3V3 #PWR050
 U 1 1 58FFF5CC
 P 7500 5050
-F 0 "#PWR052" H 7500 4900 50  0001 C CNN
+F 0 "#PWR050" H 7500 4900 50  0001 C CNN
 F 1 "+3V3" H 7500 5190 50  0000 C CNN
 F 2 "" H 7500 5050 50  0000 C CNN
@@
 $EndComp
 $Comp
-L +3V3 #PWR053
+L +3V3 #PWR051
 U 1 1 58FFF5CE
 P 7300 5450
-F 0 "#PWR053" H 7300 5300 50  0001 C CNN
+F 0 "#PWR051" H 7300 5300 50  0001 C CNN
 F 1 "+3V3" H 7300 5590 50  0000 C CNN
 F 2 "" H 7300 5450 50  0000 C CNN
@@
 	4300 2000 4250 2000
 $Comp
-L +3V3 #PWR054
+L +3V3 #PWR052
 U 1 1 58FFF5DB
 P 9050 3400
-F 0 "#PWR054" H 9050 3250 50  0001 C CNN
+F 0 "#PWR052" H 9050 3250 50  0001 C CNN
 F 1 "+3V3" H 9050 3540 50  0000 C CNN
 F 2 "" H 9050 3400 50  0000 C CNN
@@
 $EndComp
 $Comp
-L +3V3 #PWR055
+L +3V3 #PWR053
 U 1 1 587EE3E4
 P 8550 1900
-F 0 "#PWR055" H 8550 1750 50  0001 C CNN
+F 0 "#PWR053" H 8550 1750 50  0001 C CNN
 F 1 "+3V3" H 8550 2040 50  0000 C CNN
 F 2 "" H 8550 1900 50  0000 C CNN

Commit message: [mainboard] first traces routed, some pins in schematic swapped
Parts:
- removed R502: 2k00, Resistors_THT:R_Axial_DIN0204_L3.6mm_D1.6mm_P5.08mm_Horizontal, symbol R
Changed lines of the file:
@@
-$EndComp
-$Comp
-L R R502
-U 1 1 587AF381
-P 4450 2200
-F 0 "R502" V 4350 2200 50  0000 C CNN
-F 1 "2k00" V 4450 2200 50  0000 C CNN
-F 2 "Resistors_THT:R_Axial_DIN0204_L3.6mm_D1.6mm_P5.08mm_Horizontal" V 4380 2200 50  0001 C CNN
-F 3 "" H 4450 2200 50  0000 C CNN
-	1    4450 2200
-	0    1    1    0
 $EndComp
 $Comp
@@
 Wire Wire Line
 	9050 3400 8950 3400
-Wire Wire Line
-	4250 2200 4300 2200
 Text HLabel 4200 2400 0    60   Input ~ 0
 RTD1_B
