File: boards/pi-board/pi-board.sch (KiCad schematic (older format))
At the start: 12 parts, among them J1 Camera lense heater, J2 Main / Powerboard, J3 USB_A, J4 Camera light board, J5 Flir lepton board, Q1 Q_PMOS_GDS

Commit message: board/pi: schematics: cleanup, bugfixing, added power LED and testpoints
Parts:
- removed J1: Camera lense heater, symbol CONN_01X02
- removed J3: USB_A, symbol USB_A
- removed Q1: Q_PMOS_GDS, symbol Q_PMOS_GDS
- removed R1: 10k, symbol R
- added D?: LED, symbol LED
- added J?: DB9_MALE, symbol DB9_MALE
- added R?: 220R, symbol R
Connections:
- net labels removed: 28V_RXSM, Lens_heat_EN, RXSM_28V
- wire segments 166 -> 162
Other:
- note added: "red power LED"
- moved on the sheet: C1, C2, C3, C4, J2, J4, J5, MD1

Commit message: boards/pi: revise schematics - wip
Parts:
- added SW?: SW_Push, symbol SW_Push
Connections:
- net GND: now also MD1.168 (USB_OTGID), SW?.2
- net at MD1.2 (EMMC_DISABLE_N): now also SW?.1
- no-connect marks 96 -> 94
Changed lines of the file:
@@
 LIBS:valves
 LIBS:pam2306
+LIBS:switches
 LIBS:pi-board-cache
 EELAYER 25 0
@@
 $EndComp
 $Comp
-L +3.3V #PWR1
+L +3.3V #PWR01
 U 1 1 5904BC22
 P 15900 9150
-F 0 "#PWR1" H 15900 9000 50  0001 C CNN
+F 0 "#PWR01" H 15900 9000 50  0001 C CNN
 F 1 "+3.3V" H 15900 9290 50  0000 C CNN
 F 2 "" H 15900 9150 50  0001 C CNN
@@
 $EndComp
 $Comp
-L GND #PWR2
+L GND #PWR02
 U 1 1 5904BC42
 P 15900 10050
-F 0 "#PWR2" H 15900 9800 50  0001 C CNN
+F 0 "#PWR02" H 15900 9800 50  0001 C CNN
 F 1 "GND" H 15900 9900 50  0000 C CNN
 F 2 "" H 15900 10050 50  0001 C CNN
@@
 $EndComp
 $Comp
-L GND #PWR4
+L GND #PWR03
 U 1 1 5904BEC2
 P 17100 9850
-F 0 "#PWR4" H 17100 9600 50  0001 C CNN
+F 0 "#PWR03" H 17100 9600 50  0001 C CNN
 F 1 "GND" H 17100 9700 50  0000 C CNN
 F 2 "" H 17100 9850 50  0001 C CNN
@@
 $EndComp
 $Comp
-L +1V8 #PWR3
+L +1V8 #PWR04
 U 1 1 5904C298
 P 17100 9350
-F 0 "#PWR3" H 17100 9200 50  0001 C CNN
+F 0 "#PWR04" H 17100 9200 50  0001 C CNN
 F 1 "+1V8" H 17100 9490 50  0000 C CNN
 F 2 "" H 17100 9350 50  0001 C CNN
@@
 	0    -1   -1   0
 $EndComp
-NoConn ~ 17150 6800
 NoConn ~ 15200 6800
 NoConn ~ 15050 6800
@@
 NoConn ~ 6050 6800
 NoConn ~ 5900 6800
-NoConn ~ 4550 6800
 NoConn ~ 4250 6800
 NoConn ~ 4100 6800
@@
 NoConn ~ 17000 4800
 $Comp
-L GND #PWR?
+L GND #PWR05
 U 1 1 590B8C1F
 P 7350 9050
-F 0 "#PWR?" H 7350 8800 50  0001 C CNN
+F 0 "#PWR05" H 7350 8800 50  0001 C CNN
 F 1 "GND" H 7350 8900 50  0000 C CNN
 F 2 "" H 7350 9050 50  0001 C CNN
@@
 NoConn ~ 4950 9250
 $Comp
-L GND #PWR?
+L GND #PWR06
 U 1 1 590B96F8
 P 5500 9100
-F 0 "#PWR?" H 5500 8850 50  0001 C CNN
+F 0 "#PWR06" H 5500 8850 50  0001 C CNN
 F 1 "GND" H 5500 8950 50  0000 C CNN
 F 2 "" H 5500 9100 50  0001 C CNN
@@
 $EndComp
 $Comp
-L GND #PWR?
+L GND #PWR07
 U 1 1 590BC254
 P 4450 3650
-F 0 "#PWR?" H 4450 3400 50  0001 C CNN
+F 0 "#PWR07" H 4450 3400 50  0001 C CNN
 F 1 "GND" H 4450 3500 50  0000 C CNN
 F 2 "" H 4450 3650 50  0001 C CNN
@@
 $EndComp
 $Comp
-L GND #PWR?
+L GND #PWR08
 U 1 1 590BCB0F
 P 17400 4600
-F 0 "#PWR?" H 17400 4350 50  0001 C CNN
+F 0 "#PWR08" H 17400 4350 50  0001 C CNN
 F 1 "GND" H 17400 4450 50  0000 C CNN
 F 2 "" H 17400 4600 50  0001 C CNN
@@
 $EndComp
 $Comp
-L GND #PWR?
+L GND #PWR09
 U 1 1 590BCB77
 P 17400 7050
-F 0 "#PWR?" H 17400 6800 50  0001 C CNN
+F 0 "#PWR09" H 17400 6800 50  0001 C CNN
 F 1 "GND" H 17400 6900 50  0000 C CNN
 F 2 "" H 17400 7050 50  0001 C CNN
@@
 $EndComp
 $Comp
-L GND #PWR?
+L GND #PWR010
 U 1 1 590C153A
 P 6200 8850
-F 0 "#PWR?" H 6200 8600 50  0001 C CNN
+F 0 "#PWR010" H 6200 8600 50  0001 C CNN
 F 1 "GND" H 6200 8700 50  0000 C CNN
 F 2 "" H 6200 8850 50  0001 C CNN
@@
 Connection ~ 14300 4400
 Wire Wire Line
-	17600 7600 17600 4400
+	17600 4400 17600 7600
 Connection ~ 14300 7600
 Wire Wire Line
@@
 Wire Wire Line
 	6200 8700 6200 8850
-Wire Wire Line
-	1700 7600 17600 7600
 Connection ~ 2150 8450
 Wire Wire Line
@@
 	1700 4300 2750 4300
 Wire Wire Line
-	1700 4300 1700 7600
+	1700 7600 1700 4300
 Connection ~ 2600 4300
 Connection ~ 2750 7600
 Connection ~ 2600 7600
 Connection ~ 4550 8700
+Wire Wire Line
+	4550 6800 4550 7000
+Connection ~ 4550 7000
+Wire Wire Line
+	17600 7600 1700 7600
+$Comp
+L SW_Push SW?
+U 1 1 590C8968
+P 18450 6800
+F 0 "SW?" H 18500 6900 50  0000 L CNN
+F 1 "SW_Push" H 18450 6740 50  0000 C CNN
+F 2 "" H 18450 7000 50  0001 C CNN
+F 3 "" H 18450 7000 50  0001 C CNN
+	1    18450 6800
+	1    0    0    -1
+$EndComp
+Wire Wire Line
+	17150 6800 18250 6800
+$Comp
+L GND #PWR?
+U 1 1 590C8CF7
+P 18650 6950
+F 0 "#PWR?" H 18650 6700 50  0001 C CNN
+F 1 "GND" H 18650 6800 50  0000 C CNN
+F 2 "" H 18650 6950 50  0001 C CNN
+F 3 "" H 18650 6950 50  0001 C CNN
+	1    18650 6950
+	1    0    0    -1
+$EndComp
+Wire Wire Line
+	18650 6800 18650 6950
 $EndSCHEMATC

Commit message: schematics/pi: added USB boot wiring
Parts:
- removed SW?: SW_Push, symbol SW_Push
- added D?: LED, D? Gruen, symbol LED
- added J?: USB_OTG, symbol USB_OTG
- added J? (x3): GS3, Connectors:GS3, symbol GS3
- added Q? (x2): Q_NMOS_DGS, symbol Q_NMOS_DGS
- added R?: 100k, symbol R
- added R?: 47k, symbol R
- added R?: 470R, symbol R
- added TP?: TEST, symbol TEST
Connections:
- net GND: now also J?.3 (G3), J?.5 (GND), J?.6 (Shield), Q?.3 (S), R?.2
- net stepdown_pi/1V8: now also R?.2
- net at MD1.165 (USB_DP): now also J?.2 (G2); no longer J?.8
- net at MD1.167 (USB_DM): now also J?.2 (G2); no longer J?.4
- net at MD1.2 (EMMC_DISABLE_N): now also Q?.1 (D)
- net at MD1.90 (EMMC_EN_N_1V8): now also Q?.2 (G), R?.1
- net at J?.3: now also J?.3 (G3)
- new net: J?.3 (G3), J?.4
- new net: J?.1 (G1), J?.2 (D-)
- new net: J?.1 (G1), J?.3 (D+)
- new net: D?.1 (K), Q?.1 (D), Q?.3 (S)
- new net: J?.2 (G2), Q?.2 (G), R?.1
- new net: D?.2 (A), R?.2, TP?.1
- new net 3V3: R?.1
- new net VUSB: J?.1 (G1), J?.1 (VBUS)
- no-connect marks 94 -> 93
Other:
- note added: "RGB camera"
- note added: "Status ACT LED"
- note added: "USB boot"
- note added: "USB boot enable (like CMIO schematics)"
- moved on the sheet: C1, C2, C3, C4, J?

Commit message: schematics/pi: minor corrections, added annotation and most footprints
Parts:
- removed D?: LED, D? Gruen, symbol LED
- added C5: 47u, Capacitors_SMD:C_0603_HandSoldering, symbol C
- added D2: LED, LEDs:LED_0603, symbol LED
- D1: renamed from D?; footprint (none) -> LEDs:LED_0603
- J3: renamed from J?; footprint (none) -> Connectors:DB9MD
- J5: renamed from J?; footprint (none) -> Connectors:USB_Micro-B
- R1, R2, R3, R4: renamed from R?; footprint (none) -> Resistors_SMD:R_0603
- gave numbers to parts that had none: 6
- renumbered J4 to J6, J5 to J8
Connections:
- net GND: now also C5.2; no longer J2.1
- net UART_RX: now reaches MD1.51 (GPIO14)
- net UART_RX: now also J2.1
- net at J3.3: no longer J4.3 (G3)
- net at J3.8: now also J4.3 (G3)
- net at Q1.1 (D), Q2.3 (S): now also D2.1 (K)
- net at R4.2, TP1.1: now also D2.2 (A)
- new net +5V: C5.1
- no-connect marks 93 -> 99
Changed lines of the file:
@@
 Camera_light
 $Comp
-L CONN_01X04 J4
+L CONN_01X04 J6
 U 1 1 5904EE31
 P 7000 9350
-F 0 "J4" H 7000 9600 50  0000 C CNN
+F 0 "J6" H 7000 9600 50  0000 C CNN
 F 1 "Camera light board" V 7100 9350 50  0000 C CNN
 F 2 "" H 7000 9350 50  0001 C CNN
@@
 Text Label 14600 3700 0    60   ~ 0
 CLCK
-Text Label 16550 3900 0    60   ~ 0
+Text Label 16550 3950 0    60   ~ 0
 SDA
-Text Label 16400 3750 0    60   ~ 0
+Text Label 16400 3850 0    60   ~ 0
 SCL
 Text Label 15200 3650 0    60   ~ 0
 CE
 $Comp
-L CONN_01X08 J5
+L CONN_01X08 J8
 U 1 1 59071AB8
 P 14850 2900
-F 0 "J5" H 14850 3350 50  0000 C CNN
+F 0 "J8" H 14850 3350 50  0000 C CNN
 F 1 "Flir lepton board" V 14950 2900 50  0000 C CNN
 F 2 "" H 14850 2900 50  0001 C CNN
@@
 $EndComp
 $Comp
-L DB9_MALE J?
+L DB9_MALE J3
 U 1 1 590BB621
 P 4750 2600
-F 0 "J?" H 4750 3150 50  0000 C CNN
+F 0 "J3" H 4750 3150 50  0000 C CNN
 F 1 "DB9_MALE" H 4750 2025 50  0000 C CNN
-F 2 "" H 4750 2600 50  0001 C CNN
+F 2 "Connectors:DB9MD" H 4750 2600 50  0001 C CNN
 F 3 "" H 4750 2600 50  0001 C CNN
 	1    4750 2600
@@
 $EndComp
 $Comp
-L LED D?
+L LED D1
 U 1 1 590C09FF
 P 6050 8700
-F 0 "D?" H 6050 8800 50  0000 C CNN
+F 0 "D1" H 6050 8800 50  0000 C CNN
 F 1 "LED" H 6050 8600 50  0000 C CNN
-F 2 "" H 6050 8700 50  0001 C CNN
+F 2 "LEDs:LED_0603" H 6050 8700 50  0001 C CNN
 F 3 "" H 6050 8700 50  0001 C CNN
 	1    6050 8700
@@
 $EndComp
 $Comp
-L R R?
+L R R1
 U 1 1 590C0B81
 P 5550 8700
-F 0 "R?" V 5630 8700 50  0000 C CNN
+F 0 "R1" V 5630 8700 50  0000 C CNN
 F 1 "220R" V 5550 8700 50  0000 C CNN
-F 2 "" V 5480 8700 50  0001 C CNN
+F 2 "Resistors_SMD:R_0603" V 5480 8700 50  0001 C CNN
 F 3 "" H 5550 8700 50  0001 C CNN
 	1    5550 8700
@@
 red power LED
 $Comp
-L USB_OTG J?
+L USB_OTG J5
 U 1 1 590F0D7A
 P 6200 2550
-F 0 "J?" H 6000 3000 50  0000 L CNN
+F 0 "J5" H 6000 3000 50  0000 L CNN
 F 1 "USB_OTG" H 6000 2900 50  0000 L CNN
-F 2 "" H 6350 2500 50  0001 C CNN
+F 2 "Connectors:USB_Micro-B" H 6350 2500 50  0001 C CNN
 F 3 "" H 6350 2500 50  0001 C CNN
 	1    6200 2550
@@
 $EndComp
 $Comp
-L GS3 J?
+L GS3 J1
 U 1 1 590F118A
 P 4550 3700
-F 0 "J?" H 4600 3900 50  0000 C CNN
+F 0 "J1" H 4600 3900 50  0000 C CNN
 F 1 "GS3" H 4600 3501 50  0000 C CNN
 F 2 "Connectors:GS3" V 4638 3626 50  0001 C CNN
@@
 $EndComp
 $Comp
-L GS3 J?
+L GS3 J4
 U 1 1 590F124B
 P 5050 3700
-F 0 "J?" H 5100 3900 50  0000 C CNN
+F 0 "J4" H 5100 3900 50  0000 C CNN
 F 1 "GS3" H 5100 3501 50  0000 C CNN
 F 2 "Connectors:GS3" V 5138 3626 50  0001 C CNN
@@
 VUSB
 $Comp
-L GND #PWR?
+L GND #PWR011
 U 1 1 590F4D59
 P 5500 2700
-F 0 "#PWR?" H 5500 2450 50  0001 C CNN
+F 0 "#PWR011" H 5500 2450 50  0001 C CNN
 F 1 "GND" H 5500 2550 50  0000 C CNN
 F 2 "" H 5500 2700 50  0001 C CNN
@@
 $EndComp
 $Comp
-L GS3 J?
+L GS3 J7
 U 1 1 590F66C9
 P 13000 9500
-F 0 "J?" H 13050 9700 50  0000 C CNN
+F 0 "J7" H 13050 9700 50  0000 C CNN
 F 1 "GS3" H 13050 9301 50  0000 C CNN
 F 2 "Connectors:GS3" V 13088 9426 50  0001 C CNN
@@
 $EndComp
 $Comp
-L GND #PWR?
+L GND #PWR012
 U 1 1 590F6948
 P 12700 9050
-F 0 "#PWR?" H 12700 8800 50  0001 C CNN
+F 0 "#PWR012" H 12700 8800 50  0001 C CNN
 F 1 "GND" H 12700 8900 50  0000 C CNN
 F 2 "" H 12700 9050 50  0001 C CNN
@@
 VUSB
 $Comp
-L R R?
+L R R3
 U 1 1 590F779A
 P 12000 10150
-F 0 "R?" V 12080 10150 50  0000 C CNN
+F 0 "R3" V 12080 10150 50  0000 C CNN
 F 1 "47k" V 12000 10150 50  0000 C CNN
-F 2 "" V 11930 10150 50  0001 C CNN
+F 2 "Resistors_SMD:R_0603" V 11930 10150 50  0001 C CNN
 F 3 "" H 12000 10150 50  0001 C CNN
 	1    12000 10150
@@
 3V3
 $Comp
-L R R?
+L R R4
 U 1 1 590F7E93
 P 13300 11800
-F 0 "R?" V 13380 11800 50  0000 C CNN
+F 0 "R4" V 13380 11800 50  0000 C CNN
 F 1 "470R" V 13300 11800 50  0000 C CNN
-F 2 "" V 13230 11800 50  0001 C CNN
+F 2 "Resistors_SMD:R_0603" V 13230 11800 50  0001 C CNN
 F 3 "" H 13300 11800 50  0001 C CNN
 	1    13300 11800
@@
 $EndComp
 $Comp
-L LED D?
-U 1 1 590F813C
-P 12900 11800
-F 0 "D?" H 12900 11900 50  0000 C CNN
-F 1 "LED" H 12900 11700 50  0000 C CNN
-F 2 "D? Gruen" H 12900 11800 50  0001 C CNN
-F 3 "" H 12900 11800 50  0001 C CNN
-	1    12900 11800
-	1    0    0    -1
-$EndComp
-$Comp
-L TEST TP?
+L TEST TP1
 U 1 1 590F8409
 P 13100 11950
-F 0 "TP?" H 13100 12250 50  0000 C BNN
+F 0 "TP1" H 13100 12250 50  0000 C BNN
 F 1 "TEST" H 13100 12200 50  0000 C CNN
 F 2 "" H 13100 11950 50  0001 C CNN
@@
 Status ACT LED
 $Comp
-L Q_NMOS_DGS Q?
+L Q_NMOS_DGS Q1
 U 1 1 590F65BA
 P 12350 10750
-F 0 "Q?" H 12550 10800 50  0000 L CNN
+F 0 "Q1" H 12550 10800 50  0000 L CNN
 F 1 "Q_NMOS_DGS" H 12550 10700 50  0000 L CNN
 F 2 "" H 12550 10850 50  0001 C CNN
@@
 $EndComp
 $Comp
-L Q_NMOS_DGS Q?
+L Q_NMOS_DGS Q2
 U 1 1 590F6C4A
 P 13000 10750
-F 0 "Q?" H 13200 10800 50  0000 L CNN
+F 0 "Q2" H 13200 10800 50  0000 L CNN
 F 1 "Q_NMOS_DGS" H 13200 10700 50  0000 L CNN
 F 2 "" H 13200 10850 50  0001 C CNN
@@
 	13850 4600 13850 4800
 Connection ~ 14450 4600
-Wire Wire Line
-	13400 4200 13400 4800
 Connection ~ 13850 4600
 Wire Wire Line
 	12950 4600 12950 4800
-Connection ~ 13400 4600
 Wire Wire Line
 	12500 4600 12500 4800
@@
 	16700 12950 16700 12800
 Connection ~ 16500 12950
-Wire Wire Line
-	17700 12400 17700 12500
 Wire Wire Line
 	17700 12900 17700 12800
@@
 	17800 8100 17800 4200
 Wire Wire Line
-	17800 4200 13400 4200
+	17800 4200 13250 4200
 Wire Wire Line
 	4550 8300 4550 9250
@@
 	5050 4200 4700 4200
 Wire Wire Line
-	4750 2900 4750 3550
-Wire Wire Line
 	4750 3550 4950 3550
 Wire Wire Line
@@
 	12900 9000 12900 9350
 Wire Wire Line
-	13100 9350 13100 9000
-Wire Wire Line
 	13100 9000 13350 9000
 Wire Wire Line
@@
 Wire Wire Line
 	12150 10150 13000 10150
-Wire Wire Line
-	13450 11800 13800 11800
-Wire Wire Line
-	13050 11800 13150 11800
 Wire Wire Line
 	13100 11950 13100 11800
@@
 	11350 10150 11350 11000
 $Comp
-L GND #PWR?
+L GND #PWR013
 U 1 1 590F81C8
 P 11350 11000
-F 0 "#PWR?" H 11350 10750 50  0001 C CNN
+F 0 "#PWR013" H 11350 10750 50  0001 C CNN
 F 1 "GND" H 11350 10850 50  0000 C CNN
 F 2 "" H 11350 11000 50  0001 C CNN
@@
 Wire Wire Line
 	12650 10850 12650 11800
-Wire Wire Line
-	12650 11800 12750 11800
 Connection ~ 12650 10850
 Wire Wire Line
@@
 	10400 7150 10400 6800
 $Comp
-L R R?
+L R R2
 U 1 1 590F6DAC
 P 12000 9650
-F 0 "R?" V 12080 9650 50  0000 C CNN
+F 0 "R2" V 12080 9650 50  0000 C CNN
 F 1 "100k" V 12000 9650 50  0000 C CNN
-F 2 "" V 11930 9650 50  0001 C CNN
+F 2 "Resistors_SMD:R_0603" V 11930 9650 50  0001 C CNN
 F 3 "" H 12000 9650 50  0001 C CNN
 	1    12000 9650
@@
 Text Notes 4400 2350 0    60   ~ 0
 RGB camera
+Wire Wire Line
+	13400 4800 13400 4600
+Connection ~ 13400 4600
+Wire Wire Line
+	13250 4200 13250 4800
+$Comp
+L C C5
+U 1 1 591007D5
+P 18550 12650
+F 0 "C5" H 18575 12750 50  0000 L CNN
+F 1 "47u" H 18575 12550 50  0000 L CNN
+F 2 "Capacitors_SMD:C_0603_HandSoldering" H 18588 12500 50  0001 C CNN
+F 3 "" H 18550 12650 50  0001 C CNN
+	1    18550 12650
+	1    0    0    -1
+$EndComp
+$Comp
+L GND #PWR014
+U 1 1 591007DB
+P 18550 12900
+F 0 "#PWR014" H 18550 12650 50  0001 C CNN
+F 1 "GND" H 18550 12750 50  0000 C CNN
+F 2 "" H 18550 12900 50  0001 C CNN
+F 3 "" H 18550 12900 50  0001 C CNN
+	1    18550 12900
+	1    0    0    -1
+$EndComp
+$Comp
+L +5V #PWR015
+U 1 1 591007E1
+P 18550 12400
+F 0 "#PWR015" H 18550 12250 50  0001 C CNN
+F 1 "+5V" H 18550 12540 50  0000 C CNN
+F 2 "" H 18550 12400 50  0001 C CNN
+F 3 "" H 18550 12400 50  0001 C CNN
+	1    18550 12400
+	1    0    0    -1
+$EndComp
+NoConn ~ 6000 2850
+NoConn ~ 4850 2900
+NoConn ~ 4950 2900
+NoConn ~ 5050 2900
+NoConn ~ 5150 2900
+Wire Wire Line
+	4750 3550 4750 3050
+Wire Wire Line
+	4750 3050 4650 3050
+Wire Wire Line
+	4650 3050 4650 2900
+NoConn ~ 4750 2900
+Wire Wire Line
+	17700 12500 17700 12400
+Wire Wire Line
+	18550 12900 18550 12800
+Wire Wire Line
+	18550 12500 18550 12400
+Wire Wire Line
+	13800 11800 13450 11800
+Wire Wire Line
+	13100 9350 13100 9000
+$Comp
+L LED D2
+U 1 1 59105B55
+P 12900 11800
+F 0 "D2" H 12900 11900 50  0000 C CNN
+F 1 "LED" H 12900 11700 50  0000 C CNN
+F 2 "LEDs:LED_0603" H 12900 11800 50  0001 C CNN
+F 3 "" H 12900 11800 50  0001 C CNN
+	1    12900 11800
+	1    0    0    -1
+$EndComp
+Wire Wire Line
+	13050 11800 13150 11800
+Wire Wire Line
+	12650 11800 12750 11800
 $EndSCHEMATC

Commit message: schematics/pi: added missing footprints
Parts:
- MD1: footprint _ -> pi:rpi-cm
- Q1, Q2: footprint (none) -> SMD_Packages:Conn-3
Changed lines of the file:
@@
 F 0 "MD1" H 8900 -1850 50  0000 C CNN
 F 1 "Board_RPi_CM3_200pConnector" H 9650 13450 50  0000 C CNN
-F 2 "_" H 9650 5800 10  0001 C CNN
+F 2 "pi:rpi-cm" H 9650 5800 10  0001 C CNN
 F 3 "_" H 9650 5800 10  0001 C CNN
 F 4 "_" H 9650 5800 10  0001 C CNN "Manf#"
@@
 F 0 "Q1" H 12550 10800 50  0000 L CNN
 F 1 "Q_NMOS_DGS" H 12550 10700 50  0000 L CNN
-F 2 "" H 12550 10850 50  0001 C CNN
+F 2 "SMD_Packages:Conn-3" H 12550 10850 50  0001 C CNN
 F 3 "" H 12350 10750 50  0001 C CNN
 	1    12350 10750
@@
 F 0 "Q2" H 13200 10800 50  0000 L CNN
 F 1 "Q_NMOS_DGS" H 13200 10700 50  0000 L CNN
-F 2 "" H 13200 10850 50  0001 C CNN
+F 2 "SMD_Packages:Conn-3" H 13200 10850 50  0001 C CNN
 F 3 "" H 13000 10750 50  0001 C CNN
 	1    13000 10750

Commit message: schematics/pi: choose correct footprints for L and NMOS
Parts:
- J2: footprint (none) -> Connectors:DB9MD
- Q1, Q2: footprint SMD_Packages:Conn-3 -> TO_SOT_Packages_SMD:SOT-23_Handsoldering
- TP1: footprint (none) -> Measurement_Points:Measurement_Point_Round-SMD-Pad_Small
Changed lines of the file:
@@
 F 0 "J2" H 4650 10100 50  0000 C CNN
 F 1 "Main / Powerboard" H 4650 8975 50  0000 C CNN
-F 2 "" H 4650 9550 50  0001 C CNN
+F 2 "Connectors:DB9MD" H 4650 9550 50  0001 C CNN
 F 3 "" H 4650 9550 50  0001 C CNN
 	1    4650 9550
@@
 F 0 "TP1" H 13100 12250 50  0000 C BNN
 F 1 "TEST" H 13100 12200 50  0000 C CNN
-F 2 "" H 13100 11950 50  0001 C CNN
+F 2 "Measurement_Points:Measurement_Point_Round-SMD-Pad_Small" H 13100 11950 50  0001 C CNN
 F 3 "" H 13100 11950 50  0001 C CNN
 	1    13100 11950
@@
 F 0 "Q1" H 12550 10800 50  0000 L CNN
 F 1 "Q_NMOS_DGS" H 12550 10700 50  0000 L CNN
-F 2 "SMD_Packages:Conn-3" H 12550 10850 50  0001 C CNN
+F 2 "TO_SOT_Packages_SMD:SOT-23_Handsoldering" H 12550 10850 50  0001 C CNN
 F 3 "" H 12350 10750 50  0001 C CNN
 	1    12350 10750
@@
 F 0 "Q2" H 13200 10800 50  0000 L CNN
 F 1 "Q_NMOS_DGS" H 13200 10700 50  0000 L CNN
-F 2 "SMD_Packages:Conn-3" H 13200 10850 50  0001 C CNN
+F 2 "TO_SOT_Packages_SMD:SOT-23_Handsoldering" H 13200 10850 50  0001 C CNN
 F 3 "" H 13000 10750 50  0001 C CNN
 	1    13000 10750

Commit message: boards/pi: routed the connector stuff
Connections:
- net USB-: now reaches J4.2 (G2), MD1.165 (USB_DP)
- net USB+: now reaches J1.2 (G2), MD1.167 (USB_DM)
- net USB_cam+: now reaches J1.3 (G3), J3.4
- net USB_cam-: now reaches J3.8, J4.3 (G3)
- net USB_boot+: now reaches J1.1 (G1), J5.2 (D-)
- net USB_boot-: now reaches J4.1 (G1), J5.3 (D+)
