File: boards/powerboard/powerboard.sch (KiCad schematic (older format))
At the start: 35 parts, among them J101 RXSM experiment connector, J102 Powerboard <-> Mainboard, J103 Cameraboard, J104 BLDC Motor, P101 Battery, Q101 P-FET, Q102 N-FET, Q103 N-MOS, Q104 N-MOS, U101 LM1117-3.3

Commit message: [powerboard] adjust connector to mainboard
Parts:
- removed J102: Powerboard <-> Mainboard, symbol DB37_FEMALE
- added J?: Powerboard <-> Mainboard, Pin_Headers:Pin_Header_Straight_2x20_Pitch2.54mm, symbol CONN_01X40
Connections:
- net labels added: extADC_SPI_CS1, extADC_SPI_MISO, extADC_SPI_MOSI, extADC_SPI_SCK
- wire segments 235 -> 239
Changed lines of the file:
@@
 Text Label 7750 950  0    60   ~ 0
 Lens_Heat_EN
-Text Label 1900 6050 2    60   ~ 0
-Lens_Heat_EN
-Text Label 1900 5150 2    60   ~ 0
-Probe3_EN
-Text Label 1900 5050 2    60   ~ 0
-Probe2_EN
-Text Label 1900 4950 2    60   ~ 0
-Probe1_EN
-Text Label 1900 4250 2    60   ~ 0
-Motor_U_P
 Text Label 2250 5100 0    60   ~ 0
 RXSM_28V_sense
 Text Label 7200 1850 0    60   ~ 0
-Cam_Light_EN
-Text Label 1900 5950 2    60   ~ 0
 Cam_Light_EN
 Text Label 6450 2900 0    60   ~ 0
@@
 Text Label 4900 2200 2    60   ~ 0
 Charge_status
-Text Label 1900 5850 2    60   ~ 0
-Charge_status
 Text Label 2550 2750 2    47   ~ 0
 BAT_raw
 Text Label 3650 3500 2    60   ~ 0
 Boost24V_EN
-Text Label 1900 6150 2    60   ~ 0
-Boost24V_EN
 Text Label 4900 2400 2    60   ~ 0
-Charge_EN
-Text Label 1900 5750 2    60   ~ 0
 Charge_EN
 $Sheet
@@
 Text Notes 9400 1050 0    60   ~ 0
 Pin 1, 2 & 6:\nUART from mainboard
-Text Label 1900 5250 2    60   ~ 0
-extADC_SCK
-Text Label 1900 5350 2    60   ~ 0
-extADC_MOSI
-Text Label 1900 5450 2    60   ~ 0
-extADC_MISO
-Text Label 1900 5550 2    60   ~ 0
-extADC_CS
 $Comp
 L DB15_FEMALE J104
@@
 Text Label 9600 5400 0    60   ~ 0
 Encoder_B+
-Text Label 1900 6650 2    60   ~ 0
-Hall_U
-Text Label 1900 6750 2    60   ~ 0
-Hall_V
-Text Label 1900 6850 2    60   ~ 0
-Hall_W
-Text Label 1900 6350 2    60   ~ 0
-Encoder_A+
-Text Label 1900 6450 2    60   ~ 0
-Encoder_B+
 Text Label 4400 6650 0    60   ~ 0
 LO
@@
 Text Label 4400 7500 0    60   ~ 0
 RX
-Text Label 1900 6950 2    60   ~ 0
-LO
-Text Label 1900 7050 2    60   ~ 0
-SOE
-Text Label 1900 7150 2    60   ~ 0
-SODS
-Text Label 1900 7250 2    60   ~ 0
-TX
-Text Label 1900 7350 2    60   ~ 0
-RX
 Text Notes 4050 4600 0    60   ~ 0
 Heat probe connectors in sub-schematic
-$Comp
-L DB37_FEMALE J102
-U 1 1 59027E91
-P 750 5650
-F 0 "J102" H 750 7625 50  0000 C CNN
-F 1 "Powerboard <-> Mainboard" V 950 5650 50  0000 C CNN
-F 2 "" H 750 5650 50  0001 C CNN
-F 3 "" H 750 5650 50  0001 C CNN
-	1    750  5650
-	-1   0    0    -1
-$EndComp
-$Comp
-L GND #PWR101
-U 1 1 590292DE
-P 1150 7550
-F 0 "#PWR101" H 1150 7300 50  0001 C CNN
-F 1 "GND" H 1150 7400 50  0000 C CNN
-F 2 "" H 1150 7550 50  0001 C CNN
-F 3 "" H 1150 7550 50  0001 C CNN
-	1    1150 7550
-	1    0    0    -1
-$EndComp
-$Comp
-L +5V #PWR103
-U 1 1 5905088E
-P 1350 3750
-F 0 "#PWR103" H 1350 3600 50  0001 C CNN
-F 1 "+5V" H 1350 3890 50  0000 C CNN
-F 2 "" H 1350 3750 50  0000 C CNN
-F 3 "" H 1350 3750 50  0000 C CNN
-	1    1350 3750
-	1    0    0    -1
-$EndComp
 Text Label 9600 4800 0    60   ~ 0
 Brake-
@@
 $EndComp
 Text Label 8700 5000 2    60   ~ 0
-Brake_EN
-Text Label 1900 4150 2    60   ~ 0
 Brake_EN
 $Comp
@@
 	4800 7500 4400 7500
 Wire Wire Line
-	1150 3850 1150 7550
-Wire Wire Line
-	1150 7450 1050 7450
-Wire Wire Line
-	1150 3850 1050 3850
-Connection ~ 1150 7450
-Wire Wire Line
-	1050 6550 1150 6550
-Connection ~ 1150 6550
-Wire Wire Line
-	1050 5650 1150 5650
-Connection ~ 1150 5650
-Wire Wire Line
-	1350 3750 1350 4050
-Wire Wire Line
-	1350 3950 1050 3950
-Wire Wire Line
-	1350 4050 1050 4050
-Connection ~ 1350 3950
-Wire Wire Line
-	1900 7350 1050 7350
-Wire Wire Line
-	1050 7250 1900 7250
-Wire Wire Line
-	1900 7150 1050 7150
-Wire Wire Line
-	1050 7050 1900 7050
-Wire Wire Line
-	1900 6950 1050 6950
-Wire Wire Line
-	1050 6850 1900 6850
-Wire Wire Line
-	1900 6750 1050 6750
-Wire Wire Line
-	1050 6650 1900 6650
-Wire Wire Line
-	1050 6450 1900 6450
-Wire Wire Line
-	1900 6350 1050 6350
-Wire Wire Line
-	1050 6050 1900 6050
-Wire Wire Line
-	1900 5950 1050 5950
-Wire Wire Line
-	1050 5850 1900 5850
-Wire Wire Line
-	1900 5750 1050 5750
-Wire Wire Line
-	1050 5550 1900 5550
-Wire Wire Line
-	1900 5450 1050 5450
-Wire Wire Line
-	1050 5350 1900 5350
-Wire Wire Line
-	1900 5250 1050 5250
-Wire Wire Line
-	1050 5150 1900 5150
-Wire Wire Line
-	1900 5050 1050 5050
-Wire Wire Line
-	1050 4950 1900 4950
-Wire Wire Line
-	1050 4450 1900 4450
-Wire Wire Line
-	1900 4350 1050 4350
-Wire Wire Line
-	1050 4250 1900 4250
-Wire Wire Line
 	3000 3200 3000 3500
 Wire Wire Line
@@
 	9600 4600 9600 4700
 Connection ~ 9600 4700
-Wire Wire Line
-	1050 4150 1900 4150
-Wire Wire Line
-	1050 6250 1150 6250
-Connection ~ 1150 6250
-Wire Wire Line
-	1050 6150 1900 6150
-Wire Wire Line
-	1050 4850 1150 4850
-Connection ~ 1150 4850
 Wire Wire Line
 	1050 950  1150 950
@@
 Wire Wire Line
 	4000 5450 4100 5450
-Text Label 1900 4350 2    60   ~ 0
-Motor_U_N
-Text Label 1900 4450 2    60   ~ 0
-Motor_V_P
-Text Label 1900 4550 2    60   ~ 0
-Motor_V_N
-Text Label 1900 4650 2    60   ~ 0
-Motor_W_P
-Text Label 1900 4750 2    60   ~ 0
-Motor_W_N
-Wire Wire Line
-	1050 4750 1900 4750
-Wire Wire Line
-	1050 4650 1900 4650
-Wire Wire Line
-	1900 4550 1050 4550
 Text Label 7900 3100 0    60   ~ 0
 Motor_U_P
@@
 Wire Wire Line
 	4750 1200 4650 1200
+Text Label 1700 6100 2    60   ~ 0
+Lens_Heat_EN
+Text Label 1700 5000 2    60   ~ 0
+Probe3_EN
+Text Label 1700 4900 2    60   ~ 0
+Probe2_EN
+Text Label 1700 4800 2    60   ~ 0
+Probe1_EN
+Text Label 1700 5900 2    60   ~ 0
+Cam_Light_EN
+Text Label 1700 5800 2    60   ~ 0
+Charge_status
+Text Label 1700 6200 2    60   ~ 0
+Boost24V_EN
+Text Label 1700 5700 2    60   ~ 0
+Charge_EN
+Text Label 1700 7100 2    60   ~ 0
+Hall_U
+Text Label 1700 7200 2    60   ~ 0
+Hall_V
+Text Label 1700 7300 2    60   ~ 0
+Hall_W
+Text Label 1700 6800 2    60   ~ 0
+Encoder_A+
+Text Label 1700 6900 2    60   ~ 0
+Encoder_B+
+Text Label 1700 6400 2    60   ~ 0
+LO
+Text Label 1700 6500 2    60   ~ 0
+SOE
+Text Label 1700 6600 2    60   ~ 0
+SODS
+Text Label 1700 7400 2    60   ~ 0
+TX
+Text Label 1700 7500 2    60   ~ 0
+RX
+$Comp
+L GND #PWR?
+U 1 1 5919E7BC
+P 1050 7700
+F 0 "#PWR?" H 1050 7450 50  0001 C CNN
+F 1 "GND" H 1050 7550 50  0000 C CNN
+F 2 "" H 1050 7700 50  0001 C CNN
+F 3 "" H 1050 7700 50  0001 C CNN
+	1    1050 7700
+	0    -1   -1   0
+$EndComp
+$Comp
+L +5V #PWR?
+U 1 1 5919E7C2
+P 1150 3600
+F 0 "#PWR?" H 1150 3450 50  0001 C CNN
+F 1 "+5V" H 1150 3740 50  0000 C CNN
+F 2 "" H 1150 3600 50  0000 C CNN
+F 3 "" H 1150 3600 50  0000 C CNN
+	1    1150 3600
+	1    0    0    -1
+$EndComp
+Text Label 1700 4000 2    60   ~ 0
+Brake_EN
+Text Label 1700 5200 2    60   ~ 0
+extADC_SPI_SCK
+Text Label 1700 5300 2    60   ~ 0
+extADC_SPI_MISO
+Text Label 1700 5400 2    60   ~ 0
+extADC_SPI_MOSI
+Text Label 1700 5500 2    60   ~ 0
+extADC_SPI_CS1
+Text Label 1700 4100 2    60   ~ 0
+Motor_U_P
+Text Label 1700 4200 2    60   ~ 0
+Motor_U_N
+Text Label 1700 4400 2    60   ~ 0
+Motor_V_N
+Text Label 1700 4600 2    60   ~ 0
+Motor_W_N
+Text Label 1700 4300 2    60   ~ 0
+Motor_V_P
+Text Label 1700 4500 2    60   ~ 0
+Motor_W_P
+$Comp
+L CONN_01X40 J?
+U 1 1 5919E7D3
+P 650 5650
+F 0 "J?" H 650 7700 50  0000 C CNN
+F 1 "Powerboard <-> Mainboard" V 750 5650 50  0000 C CNN
+F 2 "Pin_Headers:Pin_Header_Straight_2x20_Pitch2.54mm" H 650 5650 50  0001 C CNN
+F 3 "" H 650 5650 50  0001 C CNN
+	1    650  5650
+	-1   0    0    -1
+$EndComp
+Wire Wire Line
+	950  7600 850  7600
+Wire Wire Line
+	950  3700 850  3700
+Connection ~ 950  7600
+Wire Wire Line
+	950  5600 850  5600
+Connection ~ 950  5600
+Wire Wire Line
+	1150 3600 1150 3900
+Wire Wire Line
+	1150 3800 850  3800
+Wire Wire Line
+	1150 3900 850  3900
+Connection ~ 1150 3800
+Wire Wire Line
+	1700 7500 850  7500
+Wire Wire Line
+	850  7400 1700 7400
+Wire Wire Line
+	1700 6600 850  6600
+Wire Wire Line
+	850  6500 1700 6500
+Wire Wire Line
+	1700 6400 850  6400
+Wire Wire Line
+	850  7300 1700 7300
+Wire Wire Line
+	1700 7200 850  7200
+Wire Wire Line
+	850  7100 1700 7100
+Wire Wire Line
+	850  6900 1700 6900
+Wire Wire Line
+	1700 6800 850  6800
+Wire Wire Line
+	850  6100 1700 6100
+Wire Wire Line
+	1700 5900 850  5900
+Wire Wire Line
+	850  5800 1700 5800
+Wire Wire Line
+	1700 5700 850  5700
+Wire Wire Line
+	850  5500 1700 5500
+Wire Wire Line
+	1700 5400 850  5400
+Wire Wire Line
+	850  5300 1700 5300
+Wire Wire Line
+	1700 5200 850  5200
+Wire Wire Line
+	850  5000 1700 5000
+Wire Wire Line
+	1700 4900 850  4900
+Wire Wire Line
+	850  4800 1700 4800
+Wire Wire Line
+	850  4500 1700 4500
+Wire Wire Line
+	1700 4400 850  4400
+Wire Wire Line
+	850  4300 1700 4300
+Wire Wire Line
+	850  4000 1700 4000
+Wire Wire Line
+	950  6300 850  6300
+Connection ~ 950  6300
+Wire Wire Line
+	850  6200 1700 6200
+Wire Wire Line
+	850  4700 950  4700
+Connection ~ 950  4700
+Wire Wire Line
+	850  4600 1700 4600
+Wire Wire Line
+	1700 4200 850  4200
+Wire Wire Line
+	850  4100 1700 4100
+Wire Wire Line
+	950  3700 950  7700
+Wire Wire Line
+	950  5100 850  5100
+Connection ~ 950  5100
+Wire Wire Line
+	950  6000 850  6000
+Connection ~ 950  6000
+Wire Wire Line
+	950  7000 850  7000
+Connection ~ 950  7000
+Wire Wire Line
+	950  7700 1050 7700
+Wire Wire Line
+	850  6700 950  6700
+Connection ~ 950  6700
 $EndSCHEMATC

Commit message: [powerboard] LT3757 boost converter(s) on seperate PCB, BLDC motor connector, differential encoder
Parts:
- removed D101: D, symbol D
- removed Q103: N-MOS, symbol Q_NMOS_GSD
- removed R113: 100k, symbol R
- added J?: BAT, symbol CONN_01X01
- added J?: Boost24V_EN, symbol CONN_01X01
- added J? (x3): 24V_1, symbol CONN_01X01
- added U?: DS26LV32AT, symbol DS26LV32AT
Connections:
- net labels added: Encoder_A, Encoder_A-, Encoder_B, Encoder_B-, EndSwitch
- net labels removed: Brake-, Brake_EN
- wire segments 239 -> 237
- no-connect marks 5 -> 11
Other:
- note added: "1x or 3x 24V Boost converter\non seperate PCB"
- note added: "TODO: End Switch"
- note removed: "snubber diode"
- moved on the sheet: R111

Commit message: [powerboard] add motor driver, add DRV8312 lib
Changed lines of the file:
@@
 LIBS:lt3592
 LIBS:ds26lv32at
+LIBS:drv8312
 LIBS:powerboard-cache
 EELAYER 25 0
@@
 Title "Powerboard overview"
 Date "2017-03-14"
-Rev "10"
+Rev "12"
 Comp "VIPER"
 Comment1 ""
@@
 F10 "Phase_V" O R 10050 3000 60
 F11 "Phase_W" O R 10050 3100 60
+F12 "Current" O R 10050 3300 60
 $EndSheet
 Text Label 3350 5350 0    60   ~ 0
@@
 Text Label 3650 4350 0    60   ~ 0
 Probe3_EN
+Text Label 6450 3950 2    60   ~ 0
+Probe1_Current
 Text Label 6450 4050 2    60   ~ 0
-Probe1_Current
+Probe2_Current
 Text Label 6450 4150 2    60   ~ 0
-Probe2_Current
-Text Label 6450 4250 2    60   ~ 0
 Probe3_Current
 $Sheet
@@
 	3650 4350 4200 4350
 Wire Wire Line
-	5700 4050 6450 4050
-Wire Wire Line
-	6450 4150 5700 4150
-Wire Wire Line
-	5700 4250 6450 4250
+	5700 3950 6450 3950
+Wire Wire Line
+	6450 4050 5700 4050
+Wire Wire Line
+	5700 4150 6450 4150
 Wire Wire Line
 	3350 5050 4100 5050
@@
 Text Label 1700 4000 2    60   ~ 0
 EndSwitch
+Text Label 10800 3300 2    60   ~ 0
+Motor1_Current
+Wire Wire Line
+	10050 3300 10800 3300
 $EndSCHEMATC

Commit message: [powerboard] annotate schematics
Parts:
- gave numbers to parts that had none: 7
Changed lines of the file:
@@
 $EndComp
 $Comp
-L +5V #PWR116
+L +5V #PWR119
 U 1 1 5887310D
 P 10100 1500
-F 0 "#PWR116" H 10100 1350 50  0001 C CNN
+F 0 "#PWR119" H 10100 1350 50  0001 C CNN
 F 1 "+5V" H 10100 1640 50  0000 C CNN
 F 2 "" H 10100 1500 50  0000 C CNN
@@
 $EndComp
 $Comp
-L GND #PWR114
+L GND #PWR116
 U 1 1 5887C966
 P 8750 1350
-F 0 "#PWR114" H 8750 1100 50  0001 C CNN
+F 0 "#PWR116" H 8750 1100 50  0001 C CNN
 F 1 "GND" H 8750 1200 50  0000 C CNN
 F 2 "" H 8750 1350 50  0000 C CNN
@@
 $EndComp
 $Comp
-L +3V3 #PWR113
+L +3V3 #PWR115
 U 1 1 588B5CD1
 P 8500 5700
-F 0 "#PWR113" H 8500 5550 50  0001 C CNN
+F 0 "#PWR115" H 8500 5550 50  0001 C CNN
 F 1 "+3V3" H 8500 5840 50  0000 C CNN
 F 2 "" H 8500 5700 50  0000 C CNN
@@
 $EndComp
 $Comp
-L GND #PWR102
+L GND #PWR103
 U 1 1 58CABA0F
 P 1350 3200
-F 0 "#PWR102" H 1350 2950 50  0001 C CNN
+F 0 "#PWR103" H 1350 2950 50  0001 C CNN
 F 1 "GND" H 1350 3050 50  0000 C CNN
 F 2 "" H 1350 3200 50  0000 C CNN
@@
 RXSM_28V
 $Comp
-L GND #PWR117
+L GND #PWR120
 U 1 1 58F98D85
 P 10200 2100
-F 0 "#PWR117" H 10200 1850 50  0001 C CNN
+F 0 "#PWR120" H 10200 1850 50  0001 C CNN
 F 1 "GND" H 10200 1950 50  0000 C CNN
 F 2 "" H 10200 2100 50  0001 C CNN
@@
 Hall_W
 $Comp
-L GND #PWR118
+L GND #PWR121
 U 1 1 5900FB88
 P 10350 4400
-F 0 "#PWR118" H 10350 4150 50  0001 C CNN
+F 0 "#PWR121" H 10350 4150 50  0001 C CNN
 F 1 "GND" H 10350 4250 50  0000 C CNN
 F 2 "" H 10350 4400 50  0001 C CNN
@@
 $EndComp
 $Comp
-L +5V #PWR119
+L +5V #PWR122
 U 1 1 5901160D
 P 10350 4800
-F 0 "#PWR119" H 10350 4650 50  0001 C CNN
+F 0 "#PWR122" H 10350 4650 50  0001 C CNN
 F 1 "+5V" H 10350 4940 50  0000 C CNN
 F 2 "" H 10350 4800 50  0000 C CNN
@@
 RX
 $Comp
-L GND #PWR?
+L GND #PWR101
 U 1 1 5919E7BC
 P 1050 7700
-F 0 "#PWR?" H 1050 7450 50  0001 C CNN
+F 0 "#PWR101" H 1050 7450 50  0001 C CNN
 F 1 "GND" H 1050 7550 50  0000 C CNN
 F 2 "" H 1050 7700 50  0001 C CNN
@@
 $EndComp
 $Comp
-L +5V #PWR?
+L +5V #PWR102
 U 1 1 5919E7C2
 P 1150 3600
-F 0 "#PWR?" H 1150 3450 50  0001 C CNN
+F 0 "#PWR102" H 1150 3450 50  0001 C CNN
 F 1 "+5V" H 1150 3740 50  0000 C CNN
 F 2 "" H 1150 3600 50  0000 C CNN
@@
 Motor_W_P
 $Comp
-L CONN_01X40 J?
+L CONN_01X40 J102
 U 1 1 5919E7D3
 P 650 5650
-F 0 "J?" H 650 7700 50  0000 C CNN
+F 0 "J102" H 650 7700 50  0000 C CNN
 F 1 "Powerboard <-> Mainboard" V 750 5650 50  0000 C CNN
 F 2 "Pin_Headers:Pin_Header_Straight_2x20_Pitch2.54mm" H 650 5650 50  0001 C CNN
@@
 $EndComp
 $Comp
-L CONN_01X01 J?
+L CONN_01X01 J105
 U 1 1 591A537E
 P 3300 3000
-F 0 "J?" H 3300 3100 50  0000 C CNN
+F 0 "J105" H 3300 3100 50  0000 C CNN
 F 1 "BAT" V 3400 3000 50  0000 C CNN
 F 2 "" H 3300 3000 50  0001 C CNN
@@
 $EndComp
 $Comp
-L CONN_01X01 J?
+L CONN_01X01 J106
 U 1 1 591A9664
 P 3300 3250
-F 0 "J?" H 3300 3350 50  0000 C CNN
+F 0 "J106" H 3300 3350 50  0000 C CNN
 F 1 "Boost24V_EN" H 3200 3150 50  0000 C CNN
 F 2 "" H 3300 3250 50  0001 C CNN
@@
 $EndComp
 $Comp
-L CONN_01X01 J?
+L CONN_01X01 J107
 U 1 1 591AFED2
 P 3700 3000
-F 0 "J?" H 3700 3100 50  0000 C CNN
+F 0 "J107" H 3700 3100 50  0000 C CNN
 F 1 "24V_1" V 3800 3000 50  0000 C CNN
 F 2 "" H 3700 3000 50  0001 C CNN
@@
 $EndComp
 $Comp
-L CONN_01X01 J?
+L CONN_01X01 J108
 U 1 1 591B02F7
 P 3700 3250
-F 0 "J?" H 3700 3350 50  0000 C CNN
+F 0 "J108" H 3700 3350 50  0000 C CNN
 F 1 "24V_1" V 3800 3250 50  0000 C CNN
 F 2 "" H 3700 3250 50  0001 C CNN
@@
 $EndComp
 $Comp
-L CONN_01X01 J?
+L CONN_01X01 J109
 U 1 1 591B051E
 P 3700 3500
-F 0 "J?" H 3700 3600 50  0000 C CNN
+F 0 "J109" H 3700 3600 50  0000 C CNN
 F 1 "24V_1" V 3800 3500 50  0000 C CNN
 F 2 "" H 3700 3500 50  0001 C CNN
@@
 1x or 3x 24V Boost converter\non seperate PCB
 $Comp
-L GND #PWR?
+L GND #PWR123
 U 1 1 591C869D
 P 10350 4900
-F 0 "#PWR?" H 10350 4650 50  0001 C CNN
+F 0 "#PWR123" H 10350 4650 50  0001 C CNN
 F 1 "GND" H 10350 4750 50  0000 C CNN
 F 2 "" H 10350 4900 50  0001 C CNN
@@
 $EndComp
 $Comp
-L +5V #PWR?
+L +5V #PWR124
 U 1 1 591C9070
 P 10350 5400
-F 0 "#PWR?" H 10350 5250 50  0001 C CNN
+F 0 "#PWR124" H 10350 5250 50  0001 C CNN
 F 1 "+5V" H 10350 5540 50  0000 C CNN
 F 2 "" H 10350 5400 50  0000 C CNN
@@
 TODO: End Switch
 $Comp
-L DS26LV32AT U?
+L DS26LV32AT U102
 U 1 1 591E6770
 P 8600 4850
-F 0 "U?" H 8600 4300 60  0000 C CNN
+F 0 "U102" H 8600 4300 60  0000 C CNN
 F 1 "DS26LV32AT" H 8600 5400 60  0000 C CNN
 F 2 "" H 8700 4650 60  0001 C CNN
@@
 NoConn ~ 9100 4600
 $Comp
-L +3V3 #PWR?
+L +3V3 #PWR118
 U 1 1 591EC273
 P 9200 4500
-F 0 "#PWR?" H 9200 4350 50  0001 C CNN
+F 0 "#PWR118" H 9200 4350 50  0001 C CNN
 F 1 "+3V3" H 9200 4640 50  0000 C CNN
 F 2 "" H 9200 4500 50  0000 C CNN
@@
 $EndComp
 $Comp
-L GND #PWR?
+L GND #PWR117
 U 1 1 591EC48E
 P 9200 4300
-F 0 "#PWR?" H 9200 4050 50  0001 C CNN
+F 0 "#PWR117" H 9200 4050 50  0001 C CNN
 F 1 "GND" H 9200 4150 50  0000 C CNN
 F 2 "" H 9200 4300 50  0001 C CNN
@@
 	9100 4500 9200 4500
 $Comp
-L GND #PWR?
+L GND #PWR113
 U 1 1 591ECCC7
 P 8000 4300
-F 0 "#PWR?" H 8000 4050 50  0001 C CNN
+F 0 "#PWR113" H 8000 4050 50  0001 C CNN
 F 1 "GND" H 8000 4150 50  0000 C CNN
 F 2 "" H 8000 4300 50  0001 C CNN
@@
 	8000 4400 8100 4400
 $Comp
-L +3V3 #PWR?
+L +3V3 #PWR114
 U 1 1 591ED0E6
 P 8000 4500
-F 0 "#PWR?" H 8000 4350 50  0001 C CNN
+F 0 "#PWR114" H 8000 4350 50  0001 C CNN
 F 1 "+3V3" H 8000 4640 50  0000 C CNN
 F 2 "" H 8000 4500 50  0000 C CNN
