File: boards/powerboard/powerboard_adc_filter.sch (KiCad schematic (older format))
At the start: 34 parts, among them U1101 LMV324, U1102 LMV324

Commit message: [powerboard] BLDC motor controller
Parts:
- C1101, C1102, C1103, C1104, C1105, C1106, C1107, C1108, C1109, C1110, C1111, C1112, C1113, C1114, C1115, C1116: footprint (none) -> Capacitors_SMD:C_0603
- R1101, R1102, R1103, R1104, R1105, R1106, R1107, R1108, R1109, R1110, R1111, R1112, R1113, R1114, R1115, R1116: footprint (none) -> Resistors_SMD:R_0603
- U1101, U1102: footprint (none) -> Housings_SSOP:TSSOP-14_4.4x5mm_Pitch0.65mm
Changed lines of the file:
@@
 LIBS:ds26lv32at
 LIBS:drv8312
+LIBS:drv8332
 LIBS:powerboard-cache
 EELAYER 25 0
@@
 F 0 "U1101" H 3400 1750 50  0000 L CNN
 F 1 "LMV324" H 3400 1350 50  0000 L CNN
-F 2 "" H 3350 1650 50  0001 C CNN
+F 2 "Housings_SSOP:TSSOP-14_4.4x5mm_Pitch0.65mm" H 3350 1650 50  0001 C CNN
 F 3 "" H 3450 1750 50  0001 C CNN
 	1    3400 1550
@@
 F 0 "U1101" H 3400 3050 50  0000 L CNN
 F 1 "LMV324" H 3400 2650 50  0000 L CNN
-F 2 "" H 3350 2950 50  0001 C CNN
+F 2 "Housings_SSOP:TSSOP-14_4.4x5mm_Pitch0.65mm" H 3350 2950 50  0001 C CNN
 F 3 "" H 3450 3050 50  0001 C CNN
 	2    3400 2850
@@
 F 0 "U1101" H 3400 4350 50  0000 L CNN
 F 1 "LMV324" H 3400 3950 50  0000 L CNN
-F 2 "" H 3350 4250 50  0001 C CNN
+F 2 "Housings_SSOP:TSSOP-14_4.4x5mm_Pitch0.65mm" H 3350 4250 50  0001 C CNN
 F 3 "" H 3450 4350 50  0001 C CNN
 	3    3400 4150
@@
 F 0 "U1101" H 3400 5650 50  0000 L CNN
 F 1 "LMV324" H 3400 5250 50  0000 L CNN
-F 2 "" H 3350 5550 50  0001 C CNN
+F 2 "Housings_SSOP:TSSOP-14_4.4x5mm_Pitch0.65mm" H 3350 5550 50  0001 C CNN
 F 3 "" H 3450 5650 50  0001 C CNN
 	4    3400 5450
@@
 F 0 "R1105" V 2730 1450 50  0000 C CNN
 F 1 "47k" V 2650 1450 50  0000 C CNN
-F 2 "" V 2580 1450 50  0001 C CNN
+F 2 "Resistors_SMD:R_0603" V 2580 1450 50  0001 C CNN
 F 3 "" H 2650 1450 50  0001 C CNN
 	1    2650 1450
@@
 F 0 "R1101" V 2230 1450 50  0000 C CNN
 F 1 "47k" V 2150 1450 50  0000 C CNN
-F 2 "" V 2080 1450 50  0001 C CNN
+F 2 "Resistors_SMD:R_0603" V 2080 1450 50  0001 C CNN
 F 3 "" H 2150 1450 50  0001 C CNN
 	1    2150 1450
@@
 F 0 "C1101" H 2750 1800 50  0000 L CNN
 F 1 "220n" H 2700 1600 50  0000 L CNN
-F 2 "" H 2938 1550 50  0001 C CNN
+F 2 "Capacitors_SMD:C_0603" H 2938 1550 50  0001 C CNN
 F 3 "" H 2900 1700 50  0001 C CNN
 	1    2900 1700
@@
 F 0 "C1105" V 3250 1100 50  0000 L CNN
 F 1 "220n" V 3250 800 50  0000 L CNN
-F 2 "" H 3338 900 50  0001 C CNN
+F 2 "Capacitors_SMD:C_0603" H 3338 900 50  0001 C CNN
 F 3 "" H 3300 1050 50  0001 C CNN
 	1    3300 1050
@@
 F 0 "R1106" V 2730 2750 50  0000 C CNN
 F 1 "47k" V 2650 2750 50  0000 C CNN
-F 2 "" V 2580 2750 50  0001 C CNN
+F 2 "Resistors_SMD:R_0603" V 2580 2750 50  0001 C CNN
 F 3 "" H 2650 2750 50  0001 C CNN
 	1    2650 2750
@@
 F 0 "R1102" V 2230 2750 50  0000 C CNN
 F 1 "47k" V 2150 2750 50  0000 C CNN
-F 2 "" V 2080 2750 50  0001 C CNN
+F 2 "Resistors_SMD:R_0603" V 2080 2750 50  0001 C CNN
 F 3 "" H 2150 2750 50  0001 C CNN
 	1    2150 2750
@@
 F 0 "C1102" H 2750 3100 50  0000 L CNN
 F 1 "220n" H 2700 2900 50  0000 L CNN
-F 2 "" H 2938 2850 50  0001 C CNN
+F 2 "Capacitors_SMD:C_0603" H 2938 2850 50  0001 C CNN
 F 3 "" H 2900 3000 50  0001 C CNN
 	1    2900 3000
@@
 F 0 "C1106" V 3250 2400 50  0000 L CNN
 F 1 "220n" V 3250 2100 50  0000 L CNN
-F 2 "" H 3338 2200 50  0001 C CNN
+F 2 "Capacitors_SMD:C_0603" H 3338 2200 50  0001 C CNN
 F 3 "" H 3300 2350 50  0001 C CNN
 	1    3300 2350
@@
 F 0 "R1107" V 2730 4050 50  0000 C CNN
 F 1 "47k" V 2650 4050 50  0000 C CNN
-F 2 "" V 2580 4050 50  0001 C CNN
+F 2 "Resistors_SMD:R_0603" V 2580 4050 50  0001 C CNN
 F 3 "" H 2650 4050 50  0001 C CNN
 	1    2650 4050
@@
 F 0 "R1103" V 2230 4050 50  0000 C CNN
 F 1 "47k" V 2150 4050 50  0000 C CNN
-F 2 "" V 2080 4050 50  0001 C CNN
+F 2 "Resistors_SMD:R_0603" V 2080 4050 50  0001 C CNN
 F 3 "" H 2150 4050 50  0001 C CNN
 	1    2150 4050
@@
 F 0 "C1103" H 2750 4400 50  0000 L CNN
 F 1 "220n" H 2700 4200 50  0000 L CNN
-F 2 "" H 2938 4150 50  0001 C CNN
+F 2 "Capacitors_SMD:C_0603" H 2938 4150 50  0001 C CNN
 F 3 "" H 2900 4300 50  0001 C CNN
 	1    2900 4300
@@
 F 0 "C1107" V 3250 3700 50  0000 L CNN
 F 1 "220n" V 3250 3400 50  0000 L CNN
-F 2 "" H 3338 3500 50  0001 C CNN
+F 2 "Capacitors_SMD:C_0603" H 3338 3500 50  0001 C CNN
 F 3 "" H 3300 3650 50  0001 C CNN
 	1    3300 3650
@@
 F 0 "R1108" V 2730 5350 50  0000 C CNN
 F 1 "47k" V 2650 5350 50  0000 C CNN
-F 2 "" V 2580 5350 50  0001 C CNN
+F 2 "Resistors_SMD:R_0603" V 2580 5350 50  0001 C CNN
 F 3 "" H 2650 5350 50  0001 C CNN
 	1    2650 5350
@@
 F 0 "R1104" V 2230 5350 50  0000 C CNN
 F 1 "47k" V 2150 5350 50  0000 C CNN
-F 2 "" V 2080 5350 50  0001 C CNN
+F 2 "Resistors_SMD:R_0603" V 2080 5350 50  0001 C CNN
 F 3 "" H 2150 5350 50  0001 C CNN
 	1    2150 5350
@@
 F 0 "C1104" H 2750 5700 50  0000 L CNN
 F 1 "220n" H 2700 5500 50  0000 L CNN
-F 2 "" H 2938 5450 50  0001 C CNN
+F 2 "Capacitors_SMD:C_0603" H 2938 5450 50  0001 C CNN
 F 3 "" H 2900 5600 50  0001 C CNN
 	1    2900 5600
@@
 F 0 "C1108" V 3250 5000 50  0000 L CNN
 F 1 "220n" V 3250 4700 50  0000 L CNN
-F 2 "" H 3338 4800 50  0001 C CNN
+F 2 "Capacitors_SMD:C_0603" H 3338 4800 50  0001 C CNN
 F 3 "" H 3300 4950 50  0001 C CNN
 	1    3300 4950
@@
 F 0 "U1102" H 8200 1850 50  0000 L CNN
 F 1 "LMV324" H 8200 1450 50  0000 L CNN
-F 2 "" H 8150 1750 50  0001 C CNN
+F 2 "Housings_SSOP:TSSOP-14_4.4x5mm_Pitch0.65mm" H 8150 1750 50  0001 C CNN
 F 3 "" H 8250 1850 50  0001 C CNN
 	1    8200 1650
@@
 F 0 "U1102" H 8200 3150 50  0000 L CNN
 F 1 "LMV324" H 8200 2750 50  0000 L CNN
-F 2 "" H 8150 3050 50  0001 C CNN
+F 2 "Housings_SSOP:TSSOP-14_4.4x5mm_Pitch0.65mm" H 8150 3050 50  0001 C CNN
 F 3 "" H 8250 3150 50  0001 C CNN
 	2    8200 2950
@@
 F 0 "U1102" H 8200 4450 50  0000 L CNN
 F 1 "LMV324" H 8200 4050 50  0000 L CNN
-F 2 "" H 8150 4350 50  0001 C CNN
+F 2 "Housings_SSOP:TSSOP-14_4.4x5mm_Pitch0.65mm" H 8150 4350 50  0001 C CNN
 F 3 "" H 8250 4450 50  0001 C CNN
 	3    8200 4250
@@
 F 0 "U1102" H 8200 5750 50  0000 L CNN
 F 1 "LMV324" H 8200 5350 50  0000 L CNN
-F 2 "" H 8150 5650 50  0001 C CNN
+F 2 "Housings_SSOP:TSSOP-14_4.4x5mm_Pitch0.65mm" H 8150 5650 50  0001 C CNN
 F 3 "" H 8250 5750 50  0001 C CNN
 	4    8200 5550
@@
 F 0 "R1113" V 7530 1550 50  0000 C CNN
 F 1 "47k" V 7450 1550 50  0000 C CNN
-F 2 "" V 7380 1550 50  0001 C CNN
+F 2 "Resistors_SMD:R_0603" V 7380 1550 50  0001 C CNN
 F 3 "" H 7450 1550 50  0001 C CNN
 	1    7450 1550
@@
 F 0 "R1109" V 7030 1550 50  0000 C CNN
 F 1 "47k" V 6950 1550 50  0000 C CNN
-F 2 "" V 6880 1550 50  0001 C CNN
+F 2 "Resistors_SMD:R_0603" V 6880 1550 50  0001 C CNN
 F 3 "" H 6950 1550 50  0001 C CNN
 	1    6950 1550
@@
 F 0 "C1109" H 7550 1900 50  0000 L CNN
 F 1 "220n" H 7500 1700 50  0000 L CNN
-F 2 "" H 7738 1650 50  0001 C CNN
+F 2 "Capacitors_SMD:C_0603" H 7738 1650 50  0001 C CNN
 F 3 "" H 7700 1800 50  0001 C CNN
 	1    7700 1800
@@
 F 0 "C1113" V 8050 1200 50  0000 L CNN
 F 1 "220n" V 8050 900 50  0000 L CNN
-F 2 "" H 8138 1000 50  0001 C CNN
+F 2 "Capacitors_SMD:C_0603" H 8138 1000 50  0001 C CNN
 F 3 "" H 8100 1150 50  0001 C CNN
 	1    8100 1150
@@
 F 0 "R1114" V 7530 2850 50  0000 C CNN
 F 1 "47k" V 7450 2850 50  0000 C CNN
-F 2 "" V 7380 2850 50  0001 C CNN
+F 2 "Resistors_SMD:R_0603" V 7380 2850 50  0001 C CNN
 F 3 "" H 7450 2850 50  0001 C CNN
 	1    7450 2850
@@
 F 0 "R1110" V 7030 2850 50  0000 C CNN
 F 1 "47k" V 6950 2850 50  0000 C CNN
-F 2 "" V 6880 2850 50  0001 C CNN
+F 2 "Resistors_SMD:R_0603" V 6880 2850 50  0001 C CNN
 F 3 "" H 6950 2850 50  0001 C CNN
 	1    6950 2850
@@
 F 0 "C1110" H 7550 3200 50  0000 L CNN
 F 1 "220n" H 7500 3000 50  0000 L CNN
-F 2 "" H 7738 2950 50  0001 C CNN
+F 2 "Capacitors_SMD:C_0603" H 7738 2950 50  0001 C CNN
 F 3 "" H 7700 3100 50  0001 C CNN
 	1    7700 3100
@@
 F 0 "C1114" V 8050 2500 50  0000 L CNN
 F 1 "220n" V 8050 2200 50  0000 L CNN
-F 2 "" H 8138 2300 50  0001 C CNN
+F 2 "Capacitors_SMD:C_0603" H 8138 2300 50  0001 C CNN
 F 3 "" H 8100 2450 50  0001 C CNN
 	1    8100 2450
@@
 F 0 "R1115" V 7530 4150 50  0000 C CNN
 F 1 "47k" V 7450 4150 50  0000 C CNN
-F 2 "" V 7380 4150 50  0001 C CNN
+F 2 "Resistors_SMD:R_0603" V 7380 4150 50  0001 C CNN
 F 3 "" H 7450 4150 50  0001 C CNN
 	1    7450 4150
@@
 F 0 "R1111" V 7030 4150 50  0000 C CNN
 F 1 "47k" V 6950 4150 50  0000 C CNN
-F 2 "" V 6880 4150 50  0001 C CNN
+F 2 "Resistors_SMD:R_0603" V 6880 4150 50  0001 C CNN
 F 3 "" H 6950 4150 50  0001 C CNN
 	1    6950 4150
@@
 F 0 "C1111" H 7550 4500 50  0000 L CNN
 F 1 "220n" H 7500 4300 50  0000 L CNN
-F 2 "" H 7738 4250 50  0001 C CNN
+F 2 "Capacitors_SMD:C_0603" H 7738 4250 50  0001 C CNN
 F 3 "" H 7700 4400 50  0001 C CNN
 	1    7700 4400
@@
 F 0 "C1115" V 8050 3800 50  0000 L CNN
 F 1 "220n" V 8050 3500 50  0000 L CNN
-F 2 "" H 8138 3600 50  0001 C CNN
+F 2 "Capacitors_SMD:C_0603" H 8138 3600 50  0001 C CNN
 F 3 "" H 8100 3750 50  0001 C CNN
 	1    8100 3750
@@
 F 0 "R1116" V 7530 5450 50  0000 C CNN
 F 1 "47k" V 7450 5450 50  0000 C CNN
-F 2 "" V 7380 5450 50  0001 C CNN
+F 2 "Resistors_SMD:R_0603" V 7380 5450 50  0001 C CNN
 F 3 "" H 7450 5450 50  0001 C CNN
 	1    7450 5450
@@
 F 0 "R1112" V 7030 5450 50  0000 C CNN
 F 1 "47k" V 6950 5450 50  0000 C CNN
-F 2 "" V 6880 5450 50  0001 C CNN
+F 2 "Resistors_SMD:R_0603" V 6880 5450 50  0001 C CNN
 F 3 "" H 6950 5450 50  0001 C CNN
 	1    6950 5450
@@
 F 0 "C1112" H 7550 5800 50  0000 L CNN
 F 1 "220n" H 7500 5600 50  0000 L CNN
-F 2 "" H 7738 5550 50  0001 C CNN
+F 2 "Capacitors_SMD:C_0603" H 7738 5550 50  0001 C CNN
 F 3 "" H 7700 5700 50  0001 C CNN
 	1    7700 5700
@@
 F 0 "C1116" V 8050 5100 50  0000 L CNN
 F 1 "220n" V 8050 4800 50  0000 L CNN
-F 2 "" H 8138 4900 50  0001 C CNN
+F 2 "Capacitors_SMD:C_0603" H 8138 4900 50  0001 C CNN
 F 3 "" H 8100 5050 50  0001 C CNN
 	1    8100 5050
