File: boards/temperature-sensor/temperature-sensor-DS1731.sch (KiCad schematic (older format))
At the start: 6 parts, among them J1 CONN_01X04_MALE, U1 DS1731U

Commit message: fix/ds1731: updated footprint and dimensions, pls check footprint
Parts:
- U1: footprint Housings_SOIC:SOIC-8-1EP_3.9x4.9mm_Pitch1.27mm -> Housings_SSOP:MSOP-8_3x3mm_Pitch0.65mm
Changed lines of the file:
@@
 F 0 "U1" H 2200 2050 50  0000 C CNN
 F 1 "DS1731U" H 2150 1450 50  0000 L CNN
-F 2 "Housings_SOIC:SOIC-8-1EP_3.9x4.9mm_Pitch1.27mm" H 2250 1700 50  0001 C CNN
+F 2 "Housings_SSOP:MSOP-8_3x3mm_Pitch0.65mm" H 2250 1700 50  0001 C CNN
 F 3 "" H 2350 1800 50  0001 C CNN
 	1    2350 1700
