File: boards/CupolaFeedthrough/CupolaFeedthrough.sch (KiCad schematic (older format))
At the start: 36 parts, among them J101 CONN_01X15, J102 CONN_01X15, J103 CONN_01X15, J104 DB15_FEMALE, J105 DB15_FEMALE, J106 DB15_FEMALE, J107 GND, J108 GND, J109 GND, J110 GND, J111 GND, J112 GND, J113 GND, J114 GND, J115 GND, J116 GND, J117 GND, J118 GND, J119 GND, J120 GND, J121 GND, J122 GND, J123 GND, J124 GND, J125 GND, J126 GND, J127 GND, J128 GND, J129 GND, J130 GND, J131 GND, J132 GND, J133 GND, J134 GND, J135 GND, J136 GND

Commit message: [CupolaFeedthrough] update schematic and board
Parts:
- J107, J108, J109, J110, J111, J112, J113, J114, J115, J116, J117, J118, J119, J120, J121, J122, J123, J124, J125, J126, J127, J128, J129, J130, J131, J132, J133, J134, J135: footprint Mounting_Holes:MountingHole_3.7mm_Pad -> Mounting_Holes:MountingHole_4mm
Changed lines of the file:
@@
 LIBS:contrib
 LIBS:valves
+LIBS:CupolaFeedthrough-cache
 EELAYER 25 0
 EELAYER END
@@
 F 0 "J107" H 2100 4020 50  0000 C CNN
 F 1 "GND" H 2100 3950 50  0000 C CNN
-F 2 "Mounting_Holes:MountingHole_3.7mm_Pad" H 2300 3750 50  0001 C CNN
+F 2 "Mounting_Holes:MountingHole_4mm" H 2300 3750 50  0001 C CNN
 F 3 "" H 2300 3750 50  0001 C CNN
 	1    2100 3750
@@
 F 0 "J108" H 2300 4020 50  0000 C CNN
 F 1 "GND" H 2300 3950 50  0000 C CNN
-F 2 "Mounting_Holes:MountingHole_3.7mm_Pad" H 2500 3750 50  0001 C CNN
+F 2 "Mounting_Holes:MountingHole_4mm" H 2500 3750 50  0001 C CNN
 F 3 "" H 2500 3750 50  0001 C CNN
 	1    2300 3750
@@
 F 0 "J109" H 2500 4020 50  0000 C CNN
 F 1 "GND" H 2500 3950 50  0000 C CNN
-F 2 "Mounting_Holes:MountingHole_3.7mm_Pad" H 2700 3750 50  0001 C CNN
+F 2 "Mounting_Holes:MountingHole_4mm" H 2700 3750 50  0001 C CNN
 F 3 "" H 2700 3750 50  0001 C CNN
 	1    2500 3750
@@
 F 0 "J110" H 2700 4020 50  0000 C CNN
 F 1 "GND" H 2700 3950 50  0000 C CNN
-F 2 "Mounting_Holes:MountingHole_3.7mm_Pad" H 2900 3750 50  0001 C CNN
+F 2 "Mounting_Holes:MountingHole_4mm" H 2900 3750 50  0001 C CNN
 F 3 "" H 2900 3750 50  0001 C CNN
 	1    2700 3750
@@
 F 0 "J111" H 2900 4020 50  0000 C CNN
 F 1 "GND" H 2900 3950 50  0000 C CNN
-F 2 "Mounting_Holes:MountingHole_3.7mm_Pad" H 3100 3750 50  0001 C CNN
+F 2 "Mounting_Holes:MountingHole_4mm" H 3100 3750 50  0001 C CNN
 F 3 "" H 3100 3750 50  0001 C CNN
 	1    2900 3750
@@
 F 0 "J112" H 3100 4020 50  0000 C CNN
 F 1 "GND" H 3100 3950 50  0000 C CNN
-F 2 "Mounting_Holes:MountingHole_3.7mm_Pad" H 3300 3750 50  0001 C CNN
+F 2 "Mounting_Holes:MountingHole_4mm" H 3300 3750 50  0001 C CNN
 F 3 "" H 3300 3750 50  0001 C CNN
 	1    3100 3750
@@
 F 0 "J113" H 3300 4020 50  0000 C CNN
 F 1 "GND" H 3300 3950 50  0000 C CNN
-F 2 "Mounting_Holes:MountingHole_3.7mm_Pad" H 3500 3750 50  0001 C CNN
+F 2 "Mounting_Holes:MountingHole_4mm" H 3500 3750 50  0001 C CNN
 F 3 "" H 3500 3750 50  0001 C CNN
 	1    3300 3750
@@
 F 0 "J114" H 3500 4020 50  0000 C CNN
 F 1 "GND" H 3500 3950 50  0000 C CNN
-F 2 "Mounting_Holes:MountingHole_3.7mm_Pad" H 3700 3750 50  0001 C CNN
+F 2 "Mounting_Holes:MountingHole_4mm" H 3700 3750 50  0001 C CNN
 F 3 "" H 3700 3750 50  0001 C CNN
 	1    3500 3750
@@
 F 0 "J115" H 3700 4020 50  0000 C CNN
 F 1 "GND" H 3700 3950 50  0000 C CNN
-F 2 "Mounting_Holes:MountingHole_3.7mm_Pad" H 3900 3750 50  0001 C CNN
+F 2 "Mounting_Holes:MountingHole_4mm" H 3900 3750 50  0001 C CNN
 F 3 "" H 3900 3750 50  0001 C CNN
 	1    3700 3750
@@
 F 0 "J116" H 3900 4020 50  0000 C CNN
 F 1 "GND" H 3900 3950 50  0000 C CNN
-F 2 "Mounting_Holes:MountingHole_3.7mm_Pad" H 4100 3750 50  0001 C CNN
+F 2 "Mounting_Holes:MountingHole_4mm" H 4100 3750 50  0001 C CNN
 F 3 "" H 4100 3750 50  0001 C CNN
 	1    3900 3750
@@
 F 0 "J117" H 2100 4770 50  0000 C CNN
 F 1 "GND" H 2100 4700 50  0000 C CNN
-F 2 "Mounting_Holes:MountingHole_3.7mm_Pad" H 2300 4500 50  0001 C CNN
+F 2 "Mounting_Holes:MountingHole_4mm" H 2300 4500 50  0001 C CNN
 F 3 "" H 2300 4500 50  0001 C CNN
 	1    2100 4500
@@
 F 0 "J118" H 2300 4770 50  0000 C CNN
 F 1 "GND" H 2300 4700 50  0000 C CNN
-F 2 "Mounting_Holes:MountingHole_3.7mm_Pad" H 2500 4500 50  0001 C CNN
+F 2 "Mounting_Holes:MountingHole_4mm" H 2500 4500 50  0001 C CNN
 F 3 "" H 2500 4500 50  0001 C CNN
 	1    2300 4500
@@
 F 0 "J119" H 2500 4770 50  0000 C CNN
 F 1 "GND" H 2500 4700 50  0000 C CNN
-F 2 "Mounting_Holes:MountingHole_3.7mm_Pad" H 2700 4500 50  0001 C CNN
+F 2 "Mounting_Holes:MountingHole_4mm" H 2700 4500 50  0001 C CNN
 F 3 "" H 2700 4500 50  0001 C CNN
 	1    2500 4500
@@
 F 0 "J120" H 2700 4770 50  0000 C CNN
 F 1 "GND" H 2700 4700 50  0000 C CNN
-F 2 "Mounting_Holes:MountingHole_3.7mm_Pad" H 2900 4500 50  0001 C CNN
+F 2 "Mounting_Holes:MountingHole_4mm" H 2900 4500 50  0001 C CNN
 F 3 "" H 2900 4500 50  0001 C CNN
 	1    2700 4500
@@
 F 0 "J121" H 2900 4770 50  0000 C CNN
 F 1 "GND" H 2900 4700 50  0000 C CNN
-F 2 "Mounting_Holes:MountingHole_3.7mm_Pad" H 3100 4500 50  0001 C CNN
+F 2 "Mounting_Holes:MountingHole_4mm" H 3100 4500 50  0001 C CNN
 F 3 "" H 3100 4500 50  0001 C CNN
 	1    2900 4500
@@
 F 0 "J122" H 3100 4770 50  0000 C CNN
 F 1 "GND" H 3100 4700 50  0000 C CNN
-F 2 "Mounting_Holes:MountingHole_3.7mm_Pad" H 3300 4500 50  0001 C CNN
+F 2 "Mounting_Holes:MountingHole_4mm" H 3300 4500 50  0001 C CNN
 F 3 "" H 3300 4500 50  0001 C CNN
 	1    3100 4500
@@
 F 0 "J123" H 3300 4770 50  0000 C CNN
 F 1 "GND" H 3300 4700 50  0000 C CNN
-F 2 "Mounting_Holes:MountingHole_3.7mm_Pad" H 3500 4500 50  0001 C CNN
+F 2 "Mounting_Holes:MountingHole_4mm" H 3500 4500 50  0001 C CNN
 F 3 "" H 3500 4500 50  0001 C CNN
 	1    3300 4500
@@
 F 0 "J124" H 3500 4770 50  0000 C CNN
 F 1 "GND" H 3500 4700 50  0000 C CNN
-F 2 "Mounting_Holes:MountingHole_3.7mm_Pad" H 3700 4500 50  0001 C CNN
+F 2 "Mounting_Holes:MountingHole_4mm" H 3700 4500 50  0001 C CNN
 F 3 "" H 3700 4500 50  0001 C CNN
 	1    3500 4500
@@
 F 0 "J125" H 3700 4770 50  0000 C CNN
 F 1 "GND" H 3700 4700 50  0000 C CNN
-F 2 "Mounting_Holes:MountingHole_3.7mm_Pad" H 3900 4500 50  0001 C CNN
+F 2 "Mounting_Holes:MountingHole_4mm" H 3900 4500 50  0001 C CNN
 F 3 "" H 3900 4500 50  0001 C CNN
 	1    3700 4500
@@
 F 0 "J126" H 3900 4770 50  0000 C CNN
 F 1 "GND" H 3900 4700 50  0000 C CNN
-F 2 "Mounting_Holes:MountingHole_3.7mm_Pad" H 4100 4500 50  0001 C CNN
+F 2 "Mounting_Holes:MountingHole_4mm" H 4100 4500 50  0001 C CNN
 F 3 "" H 4100 4500 50  0001 C CNN
 	1    3900 4500
@@
 F 0 "J127" H 2100 5520 50  0000 C CNN
 F 1 "GND" H 2100 5450 50  0000 C CNN
-F 2 "Mounting_Holes:MountingHole_3.7mm_Pad" H 2300 5250 50  0001 C CNN
+F 2 "Mounting_Holes:MountingHole_4mm" H 2300 5250 50  0001 C CNN
 F 3 "" H 2300 5250 50  0001 C CNN
 	1    2100 5250
@@
 F 0 "J128" H 2300 5520 50  0000 C CNN
 F 1 "GND" H 2300 5450 50  0000 C CNN
-F 2 "Mounting_Holes:MountingHole_3.7mm_Pad" H 2500 5250 50  0001 C CNN
+F 2 "Mounting_Holes:MountingHole_4mm" H 2500 5250 50  0001 C CNN
 F 3 "" H 2500 5250 50  0001 C CNN
 	1    2300 5250
@@
 F 0 "J129" H 2500 5520 50  0000 C CNN
 F 1 "GND" H 2500 5450 50  0000 C CNN
-F 2 "Mounting_Holes:MountingHole_3.7mm_Pad" H 2700 5250 50  0001 C CNN
+F 2 "Mounting_Holes:MountingHole_4mm" H 2700 5250 50  0001 C CNN
 F 3 "" H 2700 5250 50  0001 C CNN
 	1    2500 5250
@@
 F 0 "J130" H 2700 5520 50  0000 C CNN
 F 1 "GND" H 2700 5450 50  0000 C CNN
-F 2 "Mounting_Holes:MountingHole_3.7mm_Pad" H 2900 5250 50  0001 C CNN
+F 2 "Mounting_Holes:MountingHole_4mm" H 2900 5250 50  0001 C CNN
 F 3 "" H 2900 5250 50  0001 C CNN
 	1    2700 5250
@@
 F 0 "J131" H 2900 5520 50  0000 C CNN
 F 1 "GND" H 2900 5450 50  0000 C CNN
-F 2 "Mounting_Holes:MountingHole_3.7mm_Pad" H 3100 5250 50  0001 C CNN
+F 2 "Mounting_Holes:MountingHole_4mm" H 3100 5250 50  0001 C CNN
 F 3 "" H 3100 5250 50  0001 C CNN
 	1    2900 5250
@@
 F 0 "J132" H 3100 5520 50  0000 C CNN
 F 1 "GND" H 3100 5450 50  0000 C CNN
-F 2 "Mounting_Holes:MountingHole_3.7mm_Pad" H 3300 5250 50  0001 C CNN
+F 2 "Mounting_Holes:MountingHole_4mm" H 3300 5250 50  0001 C CNN
 F 3 "" H 3300 5250 50  0001 C CNN
 	1    3100 5250
@@
 F 0 "J133" H 3300 5520 50  0000 C CNN
 F 1 "GND" H 3300 5450 50  0000 C CNN
-F 2 "Mounting_Holes:MountingHole_3.7mm_Pad" H 3500 5250 50  0001 C CNN
+F 2 "Mounting_Holes:MountingHole_4mm" H 3500 5250 50  0001 C CNN
 F 3 "" H 3500 5250 50  0001 C CNN
 	1    3300 5250
@@
 F 0 "J134" H 3500 5520 50  0000 C CNN
 F 1 "GND" H 3500 5450 50  0000 C CNN
-F 2 "Mounting_Holes:MountingHole_3.7mm_Pad" H 3700 5250 50  0001 C CNN
+F 2 "Mounting_Holes:MountingHole_4mm" H 3700 5250 50  0001 C CNN
 F 3 "" H 3700 5250 50  0001 C CNN
 	1    3500 5250
@@
 F 0 "J135" H 3700 5520 50  0000 C CNN
 F 1 "GND" H 3700 5450 50  0000 C CNN
-F 2 "Mounting_Holes:MountingHole_3.7mm_Pad" H 3900 5250 50  0001 C CNN
+F 2 "Mounting_Holes:MountingHole_4mm" H 3900 5250 50  0001 C CNN
 F 3 "" H 3900 5250 50  0001 C CNN
 	1    3700 5250
