File: boards/flir-board/flir-board.sch (KiCad schematic (older format))
At the start: 31 parts

Commit message: [flir-board] finish schematic
Parts:
- C101, C102, C103, C105, C106, C107, C108, C109, C111, C112, C113, C114, C115: renamed from C?; footprint (none) -> Capacitors_SMD:C_0603
- C104: renamed from C?; footprint (none) -> Capacitors_SMD:C_0805
- C110: renamed from C?; value 1206 -> 10u 1206; footprint (none) -> Capacitors_SMD:C_1206
- D101: renamed from D?; value D_TVS -> SMBJ3V3HE3; footprint (none) -> Diodes_SMD:D_SMB_Standard
- J101, J102: renamed from J?; footprint (none) -> Pin_Headers:Pin_Header_Straight_1x02_Pitch2.54mm
- J103: renamed from J?; footprint (none) -> Pin_Headers:Pin_Header_Straight_1x04_Pitch2.54mm
- J104: renamed from J?; footprint (none) -> Pin_Headers:Pin_Header_Straight_1x01_Pitch2.54mm
- L101: renamed from L?; footprint (none) -> Inductors_SMD:L_7.3x7.3_H3.5
- R101, R102: renamed from R?; footprint (none) -> Resistors_SMD:R_1206
- R103, R104, R105: renamed from R?; footprint (none) -> Resistors_SMD:R_0603
- U101, U102, U103: renamed from U?; footprint (none) -> TO_SOT_Packages_SMD:SOT89-5_Housing
- U104: renamed from U?; footprint (none) -> local-lib:Molex_105028-1001
- X101: renamed from X?; footprint (none) -> rleh-oscillators:xt23
Connections:
- net GND: now also U104.33 (SHIELD)
- net MOSI: now reaches J103.3 (P3), U104.11 (SPI_MOSI)
- net MISO: now reaches J103.4 (P4), U104.12 (SPI_MISO)
- net CLK: now reaches J103.2 (P2), U104.13 (SPI_CLK)
- net CS: now reaches J103.1 (P1), U104.14 (SPI_CS_L)
- net GPIO3: now reaches J104.1 (P1), U104.2 (GPIO3)
- net SCL: now reaches J102.1 (P1), U104.21 (SCL)
- net SDA: now reaches J102.2 (P2), U104.22 (SDA)
- net PWR_DWM: now reaches R104.2, U104.23 (PWR_DWN_L)
- net RESET: now reaches C111.1, R103.2, U104.24 (RESET_L)
- net CLK_25MHZ: now reaches U104.26 (MASTER_CLK), X101.3 (OUT)
- net IN_3V3: now reaches C104.1, C105.1, J101.1 (P1), L101.1, R101.1, R102.1
Other:
- note added: "Unidirectional\nTVS diode\n3.3V, V_BR=4.2V"
- moved on the sheet: C111, J102, J103, J104, R103, R104

Commit message: [flir-board] board layout
Parts:
- X101: footprint rleh-oscillators:xt23 -> rleh-oscillators:ASTMHTE
Connections:
- net +3V3: now also R102.1
- net IN_3V3: no longer R102.1
Other:
- moved on the sheet: R102
Changed lines of the file:
@@
 L +3V3 #PWR02
 U 1 1 5A051E0E
-P 5050 1300
-F 0 "#PWR02" H 5050 1150 50  0001 C CNN
-F 1 "+3V3" H 5050 1440 50  0000 C CNN
-F 2 "" H 5050 1300 50  0001 C CNN
-F 3 "" H 5050 1300 50  0001 C CNN
-	1    5050 1300
-	1    0    0    -1
-$EndComp
-Wire Wire Line
-	5050 1400 5050 1300
-Wire Wire Line
-	3800 1400 5050 1400
+P 5850 1300
+F 0 "#PWR02" H 5850 1150 50  0001 C CNN
+F 1 "+3V3" H 5850 1440 50  0000 C CNN
+F 2 "" H 5850 1300 50  0001 C CNN
+F 3 "" H 5850 1300 50  0001 C CNN
+	1    5850 1300
+	1    0    0    -1
+$EndComp
+Wire Wire Line
+	5850 1400 5850 1300
+Wire Wire Line
+	3800 1400 5850 1400
 $Comp
 L GND #PWR03
 U 1 1 5A051E4F
-P 5100 2000
-F 0 "#PWR03" H 5100 1750 50  0001 C CNN
-F 1 "GND" H 5100 1850 50  0000 C CNN
-F 2 "" H 5100 2000 50  0001 C CNN
-F 3 "" H 5100 2000 50  0001 C CNN
-	1    5100 2000
+P 5850 2000
+F 0 "#PWR03" H 5850 1750 50  0001 C CNN
+F 1 "GND" H 5850 1850 50  0000 C CNN
+F 2 "" H 5850 2000 50  0001 C CNN
+F 3 "" H 5850 2000 50  0001 C CNN
+	1    5850 2000
 	1    0    0    -1
 $EndComp
@@
 $EndComp
 Wire Wire Line
-	1950 1900 5100 1900
+	1950 1900 5850 1900
 Connection ~ 3400 1900
 $Comp
@@
 F 0 "X101" H 7500 5000 60  0000 C CNN
 F 1 "ASTMHTE-25.000MHZ-ZJ-E" H 7500 5500 51  0000 C CNN
-F 2 "rleh-oscillators:xt23" H 7500 5250 60  0001 C CNN
+F 2 "rleh-oscillators:ASTMHTE" H 7500 5250 60  0001 C CNN
 F 3 "" H 7500 5250 60  0000 C CNN
 	1    7500 5250
@@
 Connection ~ 4300 1900
 Wire Wire Line
-	5100 1900 5100 2000
+	5850 1900 5850 2000
 Connection ~ 4700 1900
 Wire Wire Line
@@
 L R R102
 U 1 1 5A0D5ECC
-P 2450 1650
-F 0 "R102" V 2530 1650 50  0000 C CNN
-F 1 "HEAT" V 2450 1650 50  0000 C CNN
-F 2 "Resistors_SMD:R_1206" V 2380 1650 50  0001 C CNN
-F 3 "" H 2450 1650 50  0001 C CNN
-	1    2450 1650
+P 5750 1650
+F 0 "R102" V 5830 1650 50  0000 C CNN
+F 1 "HEAT" V 5750 1650 50  0000 C CNN
+F 2 "Resistors_SMD:R_1206" V 5680 1650 50  0001 C CNN
+F 3 "" H 5750 1650 50  0001 C CNN
+	1    5750 1650
 	1    0    0    -1
 $EndComp
@@
 	2200 1400 2200 1500
 Connection ~ 2200 1400
-Wire Wire Line
-	2450 1500 2450 1400
-Connection ~ 2450 1400
-Wire Wire Line
-	2450 1800 2450 1900
-Connection ~ 2450 1900
 Wire Wire Line
 	2200 1800 2200 1900
@@
 IN_3V3
 $Comp
-L GND #PWR?
+L GND #PWR019
 U 1 1 5A0D0DEB
 P 9350 2950
-F 0 "#PWR?" H 9350 2700 50  0001 C CNN
+F 0 "#PWR019" H 9350 2700 50  0001 C CNN
 F 1 "GND" H 9350 2800 50  0000 C CNN
 F 2 "" H 9350 2950 50  0001 C CNN
@@
 Wire Wire Line
 	9350 2950 9250 2950
+Wire Wire Line
+	5750 1500 5750 1400
+Connection ~ 5750 1400
+Wire Wire Line
+	5750 1800 5750 1900
+Connection ~ 5750 1900
 $EndSCHEMATC
