File: boards/pixart-sensor/pixart-sensor.sch (KiCad schematic (older format))
At the start: 8 parts, among them J101 Adapter, U101 PAT9125EL

Commit message: [board][pixart-sensor] Fix sensor placement
Connections:
- wire segments 32 -> 28
Changed lines of the file:
@@
 EESchema Schematic File Version 4
+LIBS:pixart-sensor-cache
 EELAYER 26 0
 EELAYER END
@@
 L Connector:Conn_01x06_Female J101
 U 1 1 5C31006B
-P 7850 2750
-F 0 "J101" H 7878 2726 50  0000 L CNN
-F 1 "Adapter" H 7878 2635 50  0000 L CNN
-F 2 "Connector_PinHeader_2.00mm:PinHeader_1x06_P2.00mm_Vertical" H 7850 2750 50  0001 C CNN
-F 3 "~" H 7850 2750 50  0001 C CNN
-	1    7850 2750
+P 7250 2750
+F 0 "J101" H 7278 2726 50  0000 L CNN
+F 1 "Adapter" H 7278 2635 50  0000 L CNN
+F 2 "Connector_PinHeader_2.00mm:PinHeader_1x06_P2.00mm_Vertical" H 7250 2750 50  0001 C CNN
+F 3 "~" H 7250 2750 50  0001 C CNN
+	1    7250 2750
 	1    0    0    -1
 $EndComp
@@
 L power:+3V3 #PWR0103
 U 1 1 5C310164
-P 7550 2450
-F 0 "#PWR0103" H 7550 2300 50  0001 C CNN
-F 1 "+3V3" H 7565 2623 50  0000 C CNN
-F 2 "" H 7550 2450 50  0001 C CNN
-F 3 "" H 7550 2450 50  0001 C CNN
-	1    7550 2450
-	1    0    0    -1
-$EndComp
-Wire Wire Line
-	7550 2450 7550 2550
-Wire Wire Line
-	7550 2550 7650 2550
+P 6950 2450
+F 0 "#PWR0103" H 6950 2300 50  0001 C CNN
+F 1 "+3V3" H 6965 2623 50  0000 C CNN
+F 2 "" H 6950 2450 50  0001 C CNN
+F 3 "" H 6950 2450 50  0001 C CNN
+	1    6950 2450
+	1    0    0    -1
+$EndComp
+Wire Wire Line
+	6950 2450 6950 2550
+Wire Wire Line
+	6950 2550 7050 2550
 $Comp
 L power:GND #PWR0104
 U 1 1 5C31045B
-P 7450 2650
-F 0 "#PWR0104" H 7450 2400 50  0001 C CNN
-F 1 "GND" V 7455 2522 50  0000 R CNN
-F 2 "" H 7450 2650 50  0001 C CNN
-F 3 "" H 7450 2650 50  0001 C CNN
-	1    7450 2650
+P 6850 2650
+F 0 "#PWR0104" H 6850 2400 50  0001 C CNN
+F 1 "GND" V 6855 2522 50  0000 R CNN
+F 2 "" H 6850 2650 50  0001 C CNN
+F 3 "" H 6850 2650 50  0001 C CNN
+	1    6850 2650
 	0    1    1    0
 $EndComp
 Wire Wire Line
-	7450 2650 7650 2650
-Wire Wire Line
-	6150 2750 6650 2750
-Wire Wire Line
-	6150 2850 6650 2850
-Wire Wire Line
-	6150 2950 6650 2950
-Wire Wire Line
-	6150 3050 6650 3050
+	6850 2650 7050 2650
 Text Label 6650 2750 2    50   ~ 0
 ID,~CS
@@
 Text Label 6650 3050 2    50   ~ 0
 SCL,SCLK
-Text Label 7250 2750 0    50   ~ 0
-SCL,SCLK
-Text Label 7250 2850 0    50   ~ 0
-SCA,SDIO
-Text Label 7250 2950 0    50   ~ 0
-MOTION
-Text Label 7250 3050 0    50   ~ 0
-ID,~CS
-Wire Wire Line
-	7250 3050 7650 3050
-Wire Wire Line
-	7650 2950 7250 2950
-Wire Wire Line
-	7250 2850 7650 2850
-Wire Wire Line
-	7650 2750 7250 2750
 $Comp
 L Mechanical:MountingHole H101
@@
 Wire Wire Line
 	5300 4300 5300 4400
+Wire Wire Line
+	6150 2750 7050 2750
+Wire Wire Line
+	6150 2850 7050 2850
+Wire Wire Line
+	6150 2950 7050 2950
+Wire Wire Line
+	6150 3050 7050 3050
 $EndSCHEMATC

Commit message: [board][pixart-sensor] Mounting: M3 screws, distance 15mm
Parts:
- H101, H102: value M2.5 -> M3; footprint MountingHole:MountingHole_2.7mm_M2.5 -> MountingHole:MountingHole_3.2mm_M3
Changed lines of the file:
@@
 P 5800 3950
 F 0 "H101" H 5900 3996 50  0000 L CNN
-F 1 "M2.5" H 5900 3905 50  0000 L CNN
-F 2 "MountingHole:MountingHole_2.7mm_M2.5" H 5800 3950 50  0001 C CNN
+F 1 "M3" H 5900 3905 50  0000 L CNN
+F 2 "MountingHole:MountingHole_3.2mm_M3" H 5800 3950 50  0001 C CNN
 F 3 "~" H 5800 3950 50  0001 C CNN
 	1    5800 3950
@@
 P 5800 4150
 F 0 "H102" H 5900 4196 50  0000 L CNN
-F 1 "M2.5" H 5900 4105 50  0000 L CNN
-F 2 "MountingHole:MountingHole_2.7mm_M2.5" H 5800 4150 50  0001 C CNN
+F 1 "M3" H 5900 4105 50  0000 L CNN
+F 2 "MountingHole:MountingHole_3.2mm_M3" H 5800 4150 50  0001 C CNN
 F 3 "~" H 5800 4150 50  0001 C CNN
 	1    5800 4150
