File: boards/cupola-cable-board/differential_drivers.sch (KiCad schematic (older format))
At the start: 5 parts, among them IC1 AM26C31M, IC2 AM26C31M

Commit message: [boards] Swap channels for layout, add second heat resistor
Parts:
- added R8: HEAT, Resistor_SMD:R_0805_2012Metric, symbol Device:R
- C10, C11: footprint (none) -> Capacitor_SMD:C_0603_1608Metric
- IC1, IC2: footprint agg:SOIC-16 -> Package_SO:SOIC-16_3.9x9.9mm_P1.27mm
- R6: footprint (none) -> Resistor_SMD:R_0805_2012Metric
Connections:
- net +5V: now also R8.1; no longer IC1.4 (G), IC2.4 (G)
- net GND: now also R8.2
- net In0_A: now also IC1.9 (3A); no longer IC1.1 (1A)
- net In0_B: now also IC1.15 (4A); no longer IC1.7 (2A)
- net In1_A: now also IC1.1 (1A); no longer IC1.9 (3A)
- net In1_B: now also IC1.7 (2A); no longer IC1.15 (4A)
- net Out0_A: now also IC1.10 (3Y); no longer IC1.2 (1Y)
- net Out0_A*: now also IC1.11 (3Z); no longer IC1.3 (1Z)
- net Out0_B: now also IC1.14 (4Y); no longer IC1.6 (2Y)
- net Out0_B*: now also IC1.13 (4Z); no longer IC1.5 (2Z)
- net Out1_A: now also IC1.2 (1Y); no longer IC1.10 (3Y)
- net Out1_A*: now also IC1.3 (1Z); no longer IC1.11 (3Z)
- net Out1_B: now also IC1.6 (2Y); no longer IC1.14 (4Y)
- net Out1_B*: now also IC1.5 (2Z); no longer IC1.13 (4Z)
Changed lines of the file:
@@
 F 0 "C10" H 965 1096 50  0000 L CNN
 F 1 "100n" H 965 1005 50  0000 L CNN
-F 2 "" H 888 900 50  0001 C CNN
+F 2 "Capacitor_SMD:C_0603_1608Metric" H 888 900 50  0001 C CNN
 F 3 "~" H 850 1050 50  0001 C CNN
 	1    850  1050
@@
 F 0 "C11" H 1365 1096 50  0000 L CNN
 F 1 "100n" H 1365 1005 50  0000 L CNN
-F 2 "" H 1288 900 50  0001 C CNN
+F 2 "Capacitor_SMD:C_0603_1608Metric" H 1288 900 50  0001 C CNN
 F 3 "~" H 1250 1050 50  0001 C CNN
 	1    1250 1050
@@
 Wire Wire Line
 	850  1250 1050 1250
-Text HLabel 2200 1450 0    50   Input ~ 0
+Text HLabel 2200 1850 0    50   Input ~ 0
 In0_A
-Text HLabel 2200 1650 0    50   Input ~ 0
+Text HLabel 2200 2050 0    50   Input ~ 0
 In0_B
-Text HLabel 3000 850  2    50   Output ~ 0
+Text HLabel 3050 1450 2    50   Output ~ 0
 Out0_A
-Text HLabel 3000 950  2    50   Output ~ 0
+Text HLabel 3050 1550 2    50   Output ~ 0
 Out0_A*
-Text HLabel 3000 1150 2    50   Output ~ 0
+Text HLabel 3050 1750 2    50   Output ~ 0
 Out0_B
-Text HLabel 3000 1250 2    50   Output ~ 0
+Text HLabel 3050 1850 2    50   Output ~ 0
 Out0_B*
-Text HLabel 3000 1450 2    50   Output ~ 0
+Text HLabel 3050 850  2    50   Output ~ 0
 Out1_A
-Text HLabel 3000 1550 2    50   Output ~ 0
+Text HLabel 3050 950  2    50   Output ~ 0
 Out1_A*
-Text HLabel 3000 1750 2    50   Output ~ 0
+Text HLabel 3050 1150 2    50   Output ~ 0
 Out1_B
-Text HLabel 3000 1850 2    50   Output ~ 0
+Text HLabel 3050 1250 2    50   Output ~ 0
 Out1_B*
 Text HLabel 4700 850  2    50   Output ~ 0
@@
 Text HLabel 4700 1250 2    50   Output ~ 0
 Out2_B*
-Text HLabel 2200 1850 0    50   Input ~ 0
+Text HLabel 2200 1450 0    50   Input ~ 0
 In1_A
-Text HLabel 2200 2050 0    50   Input ~ 0
+Text HLabel 2200 1650 0    50   Input ~ 0
 In1_B
 Text HLabel 3850 1450 0    50   Input ~ 0
@@
 F 0 "IC1" H 2600 2275 50  0000 C CNN
 F 1 "AM26C31M" H 2600 2184 50  0000 C CNN
-F 2 "agg:SOIC-16" H 2400 650 50  0001 L CNN
+F 2 "Package_SO:SOIC-16_3.9x9.9mm_P1.27mm" H 2400 650 50  0001 L CNN
 F 3 "http://www.ti.com.cn/cn/lit/ds/symlink/am26c31.pdf" H 2400 550 50  0001 L CNN
 F 4 "4975637" H 2400 450 50  0001 L CNN "Farnell"
@@
 F 0 "IC2" H 4250 2275 50  0000 C CNN
 F 1 "AM26C31M" H 4250 2184 50  0000 C CNN
-F 2 "agg:SOIC-16" H 4050 650 50  0001 L CNN
+F 2 "Package_SO:SOIC-16_3.9x9.9mm_P1.27mm" H 4050 650 50  0001 L CNN
 F 3 "http://www.ti.com.cn/cn/lit/ds/symlink/am26c31.pdf" H 4050 550 50  0001 L CNN
 F 4 "4975637" H 4050 450 50  0001 L CNN "Farnell"
@@
 	0    -1   -1   0
 $EndComp
-$Comp
-L power:+5V #PWR036
-U 1 1 5C334668
-P 2200 1150
-F 0 "#PWR036" H 2200 1000 50  0001 C CNN
-F 1 "+5V" V 2215 1278 50  0000 L CNN
-F 2 "" H 2200 1150 50  0001 C CNN
-F 3 "" H 2200 1150 50  0001 C CNN
-	1    2200 1150
-	0    -1   -1   0
-$EndComp
 Wire Wire Line
 	2300 850  2200 850
@@
 	2300 950  2200 950
 Wire Wire Line
-	2300 1150 2200 1150
-Wire Wire Line
 	2200 1250 2300 1250
-Wire Wire Line
-	2900 850  3000 850
-Wire Wire Line
-	3000 950  2900 950
-Wire Wire Line
-	3000 1150 2900 1150
-Wire Wire Line
-	2900 1250 3000 1250
-Wire Wire Line
-	3000 1450 2900 1450
-Wire Wire Line
-	3000 1550 2900 1550
-Wire Wire Line
-	2900 1750 3000 1750
-Wire Wire Line
-	3000 1850 2900 1850
-Wire Wire Line
-	2300 1450 2200 1450
-Wire Wire Line
-	2300 1650 2200 1650
-Wire Wire Line
-	2200 1850 2300 1850
-Wire Wire Line
-	2300 2050 2200 2050
 $Comp
 L power:GND #PWR042
@@
 Wire Wire Line
 	3900 1950 3900 2050
-$Comp
-L power:+5V #PWR040
-U 1 1 5C342B58
-P 3850 1150
-F 0 "#PWR040" H 3850 1000 50  0001 C CNN
-F 1 "+5V" V 3865 1278 50  0000 L CNN
-F 2 "" H 3850 1150 50  0001 C CNN
-F 3 "" H 3850 1150 50  0001 C CNN
-	1    3850 1150
-	0    -1   -1   0
-$EndComp
 $Comp
 L power:+5V #PWR038
@@
 	3850 950  3950 950
 Wire Wire Line
-	3950 1150 3850 1150
-Wire Wire Line
 	3850 1250 3950 1250
 Wire Wire Line
@@
 F 0 "R6" H 5720 1196 50  0000 L CNN
 F 1 "HEAT" V 5650 1050 50  0000 L CNN
-F 2 "" V 5580 1150 50  0001 C CNN
+F 2 "Resistor_SMD:R_0805_2012Metric" V 5580 1150 50  0001 C CNN
 F 3 "~" H 5650 1150 50  0001 C CNN
 	1    5650 1150
@@
 Wire Wire Line
 	5650 900  5650 1000
+Wire Wire Line
+	2300 1450 2200 1450
+Wire Wire Line
+	2200 1650 2300 1650
+Wire Wire Line
+	2300 1850 2200 1850
+Wire Wire Line
+	2200 2050 2300 2050
+Wire Wire Line
+	2900 850  3050 850
+Wire Wire Line
+	3050 950  2900 950
+Wire Wire Line
+	2900 1150 3050 1150
+Wire Wire Line
+	3050 1250 2900 1250
+Wire Wire Line
+	2900 1450 3050 1450
+Wire Wire Line
+	3050 1550 2900 1550
+Wire Wire Line
+	3050 1750 2900 1750
+Wire Wire Line
+	2900 1850 3050 1850
+$Comp
+L Device:R R8
+U 1 1 5C428362
+P 6000 1150
+F 0 "R8" H 6070 1196 50  0000 L CNN
+F 1 "HEAT" V 6000 1050 50  0000 L CNN
+F 2 "Resistor_SMD:R_0805_2012Metric" V 5930 1150 50  0001 C CNN
+F 3 "~" H 6000 1150 50  0001 C CNN
+	1    6000 1150
+	1    0    0    -1
+$EndComp
+$Comp
+L power:+5V #PWR05
+U 1 1 5C428368
+P 6000 900
+F 0 "#PWR05" H 6000 750 50  0001 C CNN
+F 1 "+5V" H 6015 1073 50  0000 C CNN
+F 2 "" H 6000 900 50  0001 C CNN
+F 3 "" H 6000 900 50  0001 C CNN
+	1    6000 900
+	1    0    0    -1
+$EndComp
+$Comp
+L power:GND #PWR07
+U 1 1 5C42836E
+P 6000 1400
+F 0 "#PWR07" H 6000 1150 50  0001 C CNN
+F 1 "GND" H 6005 1227 50  0000 C CNN
+F 2 "" H 6000 1400 50  0001 C CNN
+F 3 "" H 6000 1400 50  0001 C CNN
+	1    6000 1400
+	1    0    0    -1
+$EndComp
+Wire Wire Line
+	6000 1300 6000 1400
+Wire Wire Line
+	6000 900  6000 1000
 $EndSCHEMATC
