File: boards/magnetic-distance/magnetic-distance.sch (KiCad schematic (older format))
At the start: 5 parts, among them J1 CONN_02X03, U1 DS9638, U2 AS5304

Commit message: [board][magnetic-distance] remove diff line driver, new board outline
Parts:
- removed C1: 100nF, Capacitors_SMD:C_0603_HandSoldering, symbol C
- removed J1: CONN_02X03, Pin_Headers:Pin_Header_Angled_2x03_Pitch2.54mm, symbol CONN_02X03
- removed TP1: AO, Measurement_Points:Measurement_Point_Round-SMD-Pad_Small, symbol TEST
- removed U1: DS9638, Housings_SOIC:SOIC-8_3.9x4.9mm_Pitch1.27mm, symbol DS9638
- removed U2: AS5304, Housings_SSOP:TSSOP-20_4.4x6.5mm_Pitch0.65mm, symbol AS5304
- added C101: 100n, Capacitor_SMD:C_0603_1608Metric, symbol Device:C
- added H101, H102: M2, MountingHole:MountingHole_2.2mm_M2, symbol Mechanical:MountingHole
- added J101: Cable, Connector_PinHeader_2.54mm:PinHeader_2x02_P2.54mm_Vertical, symbol Connector_Generic:Conn_02x02_Counter_Clockwise
- added R_HEAT101: 100, Resistor_SMD:R_0805_2012Metric, symbol Device:R
- added TP101: AO, TestPoint:TestPoint_THTPad_1.0x1.0mm_Drill0.5mm, symbol Connector:TestPoint
- added U101: AS5304, Package_SO:TSSOP-20_4.4x6.5mm_P0.65mm, symbol as5304:AS5304
Connections:
- net labels added: +5V
- net labels removed: A*, A_c, B*, B_c, VCC
- wire segments 37 -> 19
- no-connect marks 0 -> 1

Commit message: [board][magnetic-distance] add 10µ cap to 5V rail
Parts:
- added C102: 10µ, Capacitor_SMD:C_0603_1608Metric, symbol Device:C
Connections:
- wire segments 19 -> 21
Changed lines of the file:
@@
+	1    0    0    -1
+$EndComp
+$Comp
+L power:+5V #PWR0113
+U 1 1 5C40F3C3
+P 2150 1650
+F 0 "#PWR0113" H 2150 1500 50  0001 C CNN
+F 1 "+5V" H 2165 1823 50  0000 C CNN
+F 2 "" H 2150 1650 50  0001 C CNN
+F 3 "" H 2150 1650 50  0001 C CNN
+	1    2150 1650
+	1    0    0    -1
+$EndComp
+$Comp
+L power:GND #PWR0114
+U 1 1 5C40F3C9
+P 2150 2150
+F 0 "#PWR0114" H 2150 1900 50  0001 C CNN
+F 1 "GND" H 2155 1977 50  0000 C CNN
+F 2 "" H 2150 2150 50  0001 C CNN
+F 3 "" H 2150 2150 50  0001 C CNN
+	1    2150 2150
+	1    0    0    -1
+$EndComp
+Wire Wire Line
+	2150 2050 2150 2150
+Wire Wire Line
+	2150 1750 2150 1650
+$Comp
+L Device:C C102
+U 1 1 5C40F3D1
+P 2150 1900
+F 0 "C102" H 2265 1946 50  0000 L CNN
+F 1 "10µ" H 2265 1855 50  0000 L CNN
+F 2 "Capacitor_SMD:C_0603_1608Metric" H 2188 1750 50  0001 C CNN
+F 3 "~" H 2150 1900 50  0001 C CNN
+	1    2150 1900
 	1    0    0    -1
 $EndComp
