File: boards/batterie-connector/batterie-connector.sch (KiCad schematic (older format))
At the start: 5 parts, among them J101 2W2C, J102 +, J103 -, J104 +, J105 -

Commit message: [board][batterie-connector-board] rev2: more compact, silkscreen
Parts:
- added H101: M2.5, MountingHole:MountingHole_2.7mm_M2.5_DIN965, symbol Mechanical:MountingHole
Changed lines of the file:
@@
 EESchema Schematic File Version 4
+LIBS:batterie-connector-cache
 EELAYER 26 0
 EELAYER END
@@
 Text Label 2850 3700 0    50   ~ 0
 MINUS
+$Comp
+L Mechanical:MountingHole H101
+U 1 1 5C41F0AA
+P 5000 3650
+F 0 "H101" H 5100 3696 50  0000 L CNN
+F 1 "M2.5" H 5100 3605 50  0000 L CNN
+F 2 "MountingHole:MountingHole_2.7mm_M2.5_DIN965" H 5000 3650 50  0001 C CNN
+F 3 "~" H 5000 3650 50  0001 C CNN
+	1    5000 3650
+	1    0    0    -1
+$EndComp
 $EndSCHEMATC
