File: boards/cupola-feedthrouch-simulator/cupola-feedthrouch-simulator.kicad_pcb (KiCad board)
At the start: 2 copper layers, 134 x 107 mm, 16 parts, among them J1 DB15_Female, J10 Conn_02x15_Odd_Even, J11 Conn_02x15_Odd_Even, J12 Conn_02x15_Odd_Even, J13 Conn_02x15_Odd_Even, J15 DB25_Male_MountingHoles, J16 Conn_01x02_Male, J2 DB15_Female, J3 DB15_Female, J4 DB15_Female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

Commit message: [cupola-feedthrouch-simulator] Fix DRC issues
Routing:
- net Net-(J15-Pad0): track 0.00 -> 51.2 mm
Other:
- net class Default: clearance 0.2 -> 0.175
- rule pad_to_mask_clearance: 0.051 -> 0.1
- rule solder_mask_min_width: 0.25 -> 0.1
- rule trace_clearance: 0.2 -> 0.175
Changed lines of the file:
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@@
-(kicad_pcb (version 20171130) (host pcbnew 5.0.2-4.fc29)
+(kicad_pcb (version 20171130) (host pcbnew 5.0.0-4.fc29)
   (general
     (thickness 1.6)
     (drawings 52)
-    (tracks 686)
+    (tracks 690)
     (zones 0)
     (modules 16)
@@
     (user_trace_width 1)
     (user_trace_width 2)
-    (trace_clearance 0.2)
+    (trace_clearance 0.175)
     (zone_clearance 0.508)
     (zone_45_only no)
@@
     (pad_size 1.524 1.524)
     (pad_drill 0.762)
-    (pad_to_mask_clearance 0.051)
-    (solder_mask_min_width 0.25)
+    (pad_to_mask_clearance 0.1)
+    (solder_mask_min_width 0.1)
     (aux_axis_origin 0 0)
     (visible_elements FFFFFF7F)
@@
   (net 183 "Net-(J15-Pad0)")
   (net_class Default "This is the default net class."
-    (clearance 0.2)
+    (clearance 0.175)
     (trace_width 0.25)
     (via_dia 0.8)
@@
   (segment (start 37.999999 68.699999) (end 37.5 68.2) (width 0.25) (layer B.Cu) (net 169))
   (segment (start 89.74 141.85) (end 93.790044 137.799956) (width 0.25) (layer B.Cu) (net 169))
+  (segment (start 123.755001 145.269999) (end 125.755 143.27) (width 0.25) (layer F.Cu) (net 183))
+  (segment (start 120.775 148.25) (end 123.755001 145.269999) (width 0.25) (layer F.Cu) (net 183))
+  (segment (start 78.655 143.27) (end 83.635 148.25) (width 0.25) (layer F.Cu) (net 183))
+  (segment (start 83.635 148.25) (end 120.775 148.25) (width 0.25) (layer F.Cu) (net 183))
 )
